File: Tesi/comando 24V.sch (EAGLE design)
At the start: 63 parts, among them IC1 LM324N, IC2 LM324N, IC3 LM324N, IC4 LM324N, IC5 LM324N, IC6 LM324N, IC7 LM324N, M1_BKW_INIB AGQ20003, M1_FWD_INIB AGQ20003, M1_RUN AGQ20003, M2_BKW_INIB AGQ20003, M2_BRAKE AGQ20003, M2_FWD_INIB AGQ20003, M2_RUN AGQ20003, U1 ULN2003A, U2 ULN2003A, U3 TMP37FT9Z

Commit message: 09/03/2021
Parts:
- added J1, J2, J3, J4: 61202021621, SCARA:61202021621
Changed lines of the file:
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@@
 <part name="PROXYM_M1" library="SCARA" deviceset="CON_3F" device=""/>
 <part name="PROXYM_M2" library="SCARA" deviceset="CON_3F" device=""/>
+<part name="FRAME6" library="frames" library_urn="urn:adsk.eagle:library:229" deviceset="A4L-LOC" device=""/>
+<part name="J1" library="SCARA" deviceset="61202021621" device=""/>
+<part name="J2" library="SCARA" deviceset="61202021621" device=""/>
+<part name="J3" library="SCARA" deviceset="61202021621" device=""/>
+<part name="J4" library="SCARA" deviceset="61202021621" device=""/>
 </parts>
 <sheets>
@@
 </nets>
 </sheet>
+<sheet>
+<plain>
+</plain>
+<instances>
+<instance part="FRAME6" gate="G$1" x="0" y="0" smashed="yes">
+<attribute name="DRAWING_NAME" x="217.17" y="15.24" size="2.54" layer="94"/>
+<attribute name="LAST_DATE_TIME" x="217.17" y="10.16" size="2.286" layer="94"/>
+<attribute name="SHEET" x="230.505" y="5.08" size="2.54" layer="94"/>
+</instance>
+<instance part="J1" gate="G$1" x="63.5" y="124.46" smashed="yes" rot="R270">
+<attribute name="NAME" x="62.738" y="148.082" size="1.778" layer="95"/>
+</instance>
+<instance part="J2" gate="G$1" x="191.77" y="125.73" smashed="yes" rot="R270">
+<attribute name="NAME" x="189.738" y="149.352" size="1.778" layer="95"/>
+</instance>
+<instance part="J3" gate="G$1" x="62.23" y="44.45" smashed="yes" rot="R270">
+<attribute name="NAME" x="60.198" y="68.072" size="1.778" layer="95"/>
+</instance>
+<instance part="J4" gate="G$1" x="190.5" y="57.15" smashed="yes" rot="R270">
+<attribute name="NAME" x="189.738" y="80.772" size="1.778" layer="95"/>
+</instance>
+</instances>
+<busses>
+</busses>
+<nets>
+</nets>
+</sheet>

Commit message: 12/03/2021
Parts:
- removed IC7: LM324N, SCARA:LM324N
- removed J1, J2, J3, J4: 61202021621, SCARA:61202021621
- removed R14: 47k, SCARA:R-EU_0204/7
- removed R15: VS_5V_ADJ, SCARA:64WR5KLF
- added EN_IN_5V, U$15: STRIP_3, SCARA:STRIP_3
- added IC10, IC8: LM324N, SCARA:LM324N
- added IC9: LM324N, linear:LM324N
- added J1/J3, J4/J2, J5/J7, J8/J6: 61202021621, SCARA:61202021621
- added J10, J9, J_ARD: SBH11-PBPC-D25-ST-BK, SCARA:SBH11-PBPC-D25-ST-BK
- added U4, U5: SN74LS244N, SCARA:SN74LS244N
- IC2: device SCARA:LM324N -> linear:LM324N
- IC5: device linear:LM324N -> SCARA:LM324N
- MOT1, MOT2: value TFML-125-01-S-D -> SBH11-PBPC-D25-ST-BK; device TFML-125-01-S-D:TFML-125-01-S-D -> SCARA:SBH11-PBPC-D25-ST-BK
Connections:
- removed net IN_3V3_M1_ALM: MOT1.37
- removed net IN_3V3_M2_ALM: MOT2.37
- removed net IN_3V3_NOMING_SENS_M2: IC1B.OUT
- removed net MZ_DIR: IC6C.+IN
- removed net MZ_IMP: IC6B.+IN
- removed net MZ_TRIGGER: IC6A.+IN
- removed net VS_3V: IC1C.-IN, IC1D.-IN, IC2A.-IN, IC2B.-IN, IC2C.-IN, IC2D.-IN
- removed net VS_5V: IC4C.-IN, IC4C.OUT
- new net IN_3V3_EMRGN_CHN: J10.6, J4/J2.3
- new net IN_3V3_HOMING_SENS_M2: IC10B.OUT, J1/J3.15
- new net IN_3V3_M1_ALARM: J1/J3.19, MOT1.37
- new net IN_3V3_M2_ALARM: J4/J2.1, MOT2.37
- new net IN_3V3_SCI3_RX: J1/J3.5
- new net IN_3V3_TENS_ALARM: J9.15
- new net M1_BAT: MOT1.42
- new net N$16: U$15.2, U5.!1G, U5.!G/2G
- new net N$38: J4/J2.7
- new net N$40: J4/J2.9
- new net N$41: J4/J2.11
- new net N$43: EN_IN_5V.2, U4.!1G, U4.!G/2G
- new net N$54: J4/J2.4
- new net N$55: J4/J2.6
- new net N$56: J4/J2.18
- new net N$62: J5/J7.19
- new net N$70: J8/J6.16
- new net N$71: J8/J6.18
- new net N$83: J10.7
- new net N$84: J10.10
- new net N$85: J10.12
- new net N$88: J10.18
- new net N$89: J10.20
- new net N$92: J10.25
- new net N$93: J10.27
- new net N$94: J10.28
- new net N$96: J10.37
- new net N$97: J10.39
- new net OUT_3V3_MZ_DIR: IC5C.+IN, J8/J6.3
- new net OUT_3V3_MZ_IMP: IC5B.+IN, J8/J6.1
- new net OUT_3V3_MZ_TRIGGER: IC5A.+IN, J5/J7.17
- new net OUT_3V3_SCI_TX: J1/J3.7
- net +24V: now also IC2B.+IN, IC5P.V+, MOT1.7, MOT2.7; no longer IC4B.+IN, IC6P.V+, MOT1.07, MOT2.07, R14.2
- net +3V3: now also IC10B.-IN, IC2A.-IN, IC2B.-IN; no longer IC1B.-IN, IC4A.-IN, IC4B.-IN, IC4P.V+
- net +5V: now also EN_IN_5V.1, U$15.1, U4.VCC, U5.VCC; no longer IC7P.V+
- net 220V_PROBE: now also IC2A.+IN; no longer IC4A.+IN
- net GND: now also EN_IN_5V.3, IC5P.V-, J1/J3.4, J10.14, J10.2, J10.23, J10.32, J10.4, J4/J2.2, J5/J7.4, J8/J6.2, J9.16, J9.2, J9.25, J9.34, J9.4, MOT1.4, MOT1.6, MOT2.4, MOT2.6, U$15.3, U4.GND, U5.GND; no longer IC4P.V-, IC6P.V-, IC7P.V-, MOT1.04, MOT1.06, MOT2.04, MOT2.06, R15.1
- net IN_24V_HOMING_SENS_M2: now also IC10B.+IN; no longer IC1B.+IN
- net IN_3V3_220V_ALARM: now also IC2A.OUT; no longer IC4A.OUT
- net IN_3V3_24V_ALARM: now also IC2B.OUT; no longer IC4B.OUT
- net IN_3V3_HOMING_SENS_M1: now also J1/J3.9
- net IN_3V3_M1_ENC_PHA: now also J5/J7.13, U4.1Y1; no longer IC1C.OUT
- net IN_3V3_M1_ENC_PHB: now also J5/J7.15, U4.1Y2; no longer IC1D.OUT
- net IN_3V3_M1_ENC_PHZ: now also J5/J7.9, U4.1Y3; no longer IC2A.OUT
- net IN_3V3_M1_READY: now also J4/J2.13
- net IN_3V3_M2_ENC_PHA: now also J8/J6.4, U4.1Y4; no longer IC2B.OUT
- net IN_3V3_M2_ENC_PHB: now also J10.22, U4.2Y4; no longer IC2C.OUT
- net IN_3V3_M2_ENC_PHZ: now also J4/J2.15, U4.2Y3; no longer IC2D.OUT
- net IN_3V3_M2_READY: now also J4/J2.17
- net IN_3V3_MZ_ALARM: now also J1/J3.17
- net IN_3V3_TEMP_ALARM: now also IC8D.OUT, J4/J2.20; no longer IC3D.OUT
- net IN_5V_M1_ENC_PHA: now also U4.1A1; no longer IC1C.+IN
- net IN_5V_M1_ENC_PHB: now also U4.1A2; no longer IC1D.+IN
- net IN_5V_M1_ENC_PHZ: now also U4.1A3; no longer IC2A.+IN
- net IN_5V_M2_ENC_PHA: now also U4.1A4; no longer IC2B.+IN
- net IN_5V_M2_ENC_PHB: now also U4.2A4; no longer IC2C.+IN
- net IN_5V_M2_ENC_PHZ: now also U4.2A3; no longer IC2D.+IN
- net M2_BAT: no longer MOT1.42
- net N$14: now also IC9C.+IN; no longer IC5C.+IN
- net N$36: now also J4/J2.5; no longer IC4C.+IN, R14.1, R15.3
- net OUT_24V_M1_CCW: now also MOT1.2; no longer MOT1.02
- net OUT_24V_M1_CW: now also MOT1.1; no longer MOT1.01
- net OUT_24V_M2_CCW: now also MOT2.2; no longer MOT2.02
- net OUT_24V_M2_CW: now also MOT2.1; no longer MOT2.01
- net OUT_24V_MZ_DIR: now also IC5C.OUT; no longer IC6C.OUT
- net OUT_24V_MZ_IMP: now also IC5B.OUT; no longer IC6B.OUT
- net OUT_24V_MZ_TRIGGER: now also IC5A.OUT; no longer IC6A.OUT
- net OUT_3V3_M1_CCW: now also J8/J6.11, U5.1A2; no longer IC7B.+IN
- net OUT_3V3_M1_CW: now also J8/J6.5, U5.1A1; no longer IC7A.+IN
- net OUT_3V3_M2_CCW: now also J9.8, U5.1A4; no longer IC7D.+IN
- net OUT_3V3_M2_CW: now also J9.6, U5.1A3; no longer IC7C.+IN
- net OUT_5V_M1_CCW: now also MOT1.5, U5.1Y2; no longer IC7B.OUT, MOT1.05
- net OUT_5V_M1_CW: now also MOT1.3, U5.1Y1; no longer IC7A.OUT, MOT1.03
- net OUT_5V_M2_CCW: now also MOT2.5, U5.1Y4; no longer IC7D.OUT, MOT2.05
- net OUT_5V_M2_CW: now also MOT2.3, U5.1Y3; no longer IC7C.OUT, MOT2.03
- net OUT_M1_BKW_INIB: now also MOT1.8; no longer MOT1.08
- net OUT_M1_FWD_INIB: now also MOT1.9; no longer MOT1.09
- net OUT_M2_BKW_INIB: now also MOT2.8; no longer MOT2.08
- net OUT_M2_FWD_INIB: now also MOT2.9; no longer MOT2.09
- net TEMP: now also IC8D.+IN; no longer IC3D.+IN
- net VS_3V3: now also IC5A.-IN, IC5B.-IN, IC5C.-IN; no longer IC6A.-IN, IC6B.-IN, IC6C.-IN, IC7A.-IN, IC7B.-IN, IC7C.-IN, IC7D.-IN
- net VS_TEMP: now also IC8D.-IN, IC9C.-IN, IC9C.OUT; no longer IC3D.-IN, IC5C.-IN, IC5C.OUT

Commit message: FINE LAVORO MATTINA
Connections:
- net M1_BKW_INIB renamed OUT_5V_M1_CCW_INIB
- net M1_FWD_INIB renamed OUT_5V_M1_CW_INIB
- net M2_BKW_INIB renamed OUT_5V_M2_CCW_INIB
- net M2_FWD_INIB renamed OUT_5V_M2_CW_INIB
- removed net M1_RUN: U1.IN3
- removed net M2_RUN: U1.IN6
- removed net N$83: J10.7
- removed net N$88: J10.18
- new net IN_5V_RX: J_ARD.3
- new net N$100: J_ARD.43
- new net N$101: J_ARD.44
- new net N$102: J_ARD.45
- new net N$103: J_ARD.46
- new net N$104: J_ARD.47
- new net N$105: J_ARD.48
- new net N$106: J_ARD.49
- new net N$107: J_ARD.50
- new net N$26: J_ARD.5
- new net N$28: J_ARD.6
- new net N$30: J_ARD.7
- new net N$32: J_ARD.8
- new net N$34: J_ARD.9
- new net N$42: J_ARD.10
- new net N$44: J_ARD.11
- new net N$51: J_ARD.12
- new net N$53: J_ARD.13
- new net N$57: J_ARD.14
- new net N$58: J_ARD.15
- new net N$59: J_ARD.16
- new net N$60: J_ARD.17
- new net N$61: J_ARD.18
- new net N$63: J_ARD.19
- new net N$64: J_ARD.20
- new net N$65: J_ARD.21
- new net N$66: J_ARD.22
- new net N$67: J_ARD.23
- new net N$68: J_ARD.24
- new net N$69: J_ARD.25
- new net N$72: J_ARD.26
- new net N$73: J_ARD.27
- new net N$74: J_ARD.28
- new net N$75: J_ARD.29
- new net N$76: J_ARD.30
- new net N$77: J_ARD.31
- new net N$78: J_ARD.32
- new net N$79: J_ARD.33
- new net N$80: J_ARD.34
- new net N$81: J_ARD.35
- new net N$82: J_ARD.36
- new net N$86: J_ARD.37
- new net N$90: J_ARD.38
- new net N$91: J_ARD.39
- new net N$95: J_ARD.40
- new net N$98: J_ARD.41
- new net N$99: J_ARD.42
- new net OUT_3V3_M1_RUN: J10.7, U1.IN3
- new net OUT_3V3_M2_RUN: J10.18, U1.IN6
- new net OUT_5V_TX: J_ARD.4
- net GND: now also J_ARD.1, J_ARD.2

Commit message: pomeriggio finito
Parts:
- added EN_M1_ENC_PHZ, EN_M2_ENC_PHZ: STRIP_2, SCARA:STRIP_2
- added EN_SCI, OUT_ARD_4-7_5V-24V, OUT_ARD_8-11_5V-24V: STRIP_3, SCARA:STRIP_3
- added IC11, IC7: LM324N, SCARA:LM324N
- added J_LAMPADE: 61201021621, SCARA:61201021621
- added R14: 47k, SCARA:R-EU_0204/7
- added R15: VS_5v_ADJ, SCARA:64WR5KLF
- added SUP_3V3, SUP_5V: BR30X, SCARA:BR30X
- added U6: SN74LS244N, SCARA:SN74LS244N
- renumbered EN_IN_5V to EN_IN_ENC, U$15 to EN_OUT_MOT
Connections:
- net N$73 renamed IN_5V_GPI1_0V-30V
- net N$74 renamed IN_5V_GPI2_0V-30V
- net N$75 renamed IN_5V_GPI3_0V-30V
- net N$76 renamed IN_5V_GPI4_0V-30V
- net N$77 renamed IN_5V_GPI5_0V-30V
- net N$78 renamed IN_5V_GPI6_0V-30V
- net N$79 renamed IN_5V_GPI7_0V-30V
- net N$80 renamed IN_5V_GPI8_0V-30V
- net N$81 renamed IN_5V_GPI9_0V-30V
- net N$82 renamed IN_5V_GPI10_0V-30V
- net N$86 renamed IN_5V_GPI11_0V-30V
- removed net I/O1_24V: U2.IN2
- removed net I/O2_24V: U2.IN3
- removed net I/O3_24V: U2.IN4
- removed net I/O4_24V: U2.IN5
- removed net IN_3V3_SCI3_RX: J1/J3.5
- removed net M2_BRAKE: U1.IN7
- removed net MZ_EN: U2.IN1
- removed net N$32: J_ARD.8
- removed net N$34: J_ARD.9
- removed net N$42: J_ARD.10
- removed net N$44: J_ARD.11
- removed net N$51: J_ARD.12
- removed net N$53: J_ARD.13
- removed net N$57: J_ARD.14
- removed net N$58: J_ARD.15
- removed net N$59: J_ARD.16
- removed net N$60: J_ARD.17
- removed net N$61: J_ARD.18
- removed net N$63: J_ARD.19
- removed net N$64: J_ARD.20
- removed net N$65: J_ARD.21
- removed net N$66: J_ARD.22
- removed net N$67: J_ARD.23
- removed net N$68: J_ARD.24
- removed net N$69: J_ARD.25
- removed net N$72: J_ARD.26
- removed net N$90: J_ARD.38
- removed net N$91: J_ARD.39
- removed net N$96: J10.37
- new net IN_3V3_SCI_RX: J1/J3.5, U6.2Y4
- new net N$18: EN_SCI.2, U6.!1G, U6.!G/2G
- new net N$20: IC7D.+IN, R14.1, R15.3
- new net N$22: IC11P.V+, OUT_ARD_4-7_5V-24V.2
- new net N$24: EN_M2_ENC_PHZ.2, J4/J2.15
- new net OUT_24V-5V_GPO10: IC7C.OUT
- new net OUT_24V-5V_GPO4: IC11A.OUT
- new net OUT_24V-5V_GPO5: IC11B.OUT
- new net OUT_24V-5V_GPO6: IC11C.OUT
- new net OUT_24V-5V_GPO7: IC11D.OUT
- new net OUT_24V-5V_GPO8: IC7A.OUT
- new net OUT_24V-5V_GPO9: IC7B.OUT
- new net OUT_3V3_MZ_EN: J10.37, U2.IN1
- new net OUT_5V_GPO10_24V-5V: IC7C.+IN, J_ARD.26
- new net OUT_5V_GPO1_24V: J_ARD.17, U2.IN3
- new net OUT_5V_GPO2_24V: J_ARD.18, U2.IN4
- new net OUT_5V_GPO3_24V: J_ARD.19, U2.IN5
- new net OUT_5V_GPO4_24V-5V: IC11A.+IN, J_ARD.20
- new net OUT_5V_GPO5_24V-5V: IC11B.+IN, J_ARD.21
- new net OUT_5V_GPO6_24V-5V: IC11C.+IN, J_ARD.22
- new net OUT_5V_GPO7_24V-5V: IC11D.+IN, J_ARD.23
- new net OUT_5V_GPO8_24V-5V: IC7A.+IN, J_ARD.24
- new net OUT_5V_GPO9_24V-5V: IC7B.+IN, J_ARD.25
- new net OUT_5V_LAMPADA_1: J_ARD.12, J_LAMPADE.1
- new net OUT_5V_LAMPADA_2: J_ARD.13, J_LAMPADE.3
- new net OUT_5V_LAMPADA_3: J_ARD.14, J_LAMPADE.5
- new net OUT_5V_LAMPADA_4: J_ARD.15, J_LAMPADE.7
- new net OUT_5V_LAMPADA_5: J_ARD.16, J_LAMPADE.9
- new net OUT_5V_M2_BRAKE: J_ARD.10, U1.IN7
- new net OUT_5V_MZ_HOMING: J_ARD.11, U2.IN2
- new net VS_5V: IC11A.-IN, IC11B.-IN, IC11C.-IN, IC11D.-IN, IC7A.-IN, IC7B.-IN, IC7C.-IN, IC7D.-IN, IC7D.OUT
- net +24V: now also OUT_ARD_4-7_5V-24V.3, OUT_ARD_8-11_5V-24V.3, R14.2, SUP_3V3.VIN, SUP_5V.VIN
- net +3V3: now also SUP_3V3.VOUT
- net +5V: now also EN_SCI.1, J_ARD.3, OUT_ARD_4-7_5V-24V.1, OUT_ARD_8-11_5V-24V.1, SUP_5V.VOUT, U6.VCC
- net GND: now also EN_SCI.3, IC11P.V-, IC7P.V-, J_LAMPADE.10, J_LAMPADE.2, J_LAMPADE.4, J_LAMPADE.6, J_LAMPADE.8, R15.1, SUP_3V3.GND, SUP_5V.GND, U6.GND
- net IN_3V3_M1_ENC_PHZ: now also EN_M1_ENC_PHZ.1; no longer J5/J7.9
- net IN_3V3_M2_ENC_PHZ: now also EN_M2_ENC_PHZ.1; no longer J4/J2.15
- net IN_5V_RX: now also J_ARD.4, U6.1Y1; no longer J_ARD.3
- net N$26: now also IC7P.V+, OUT_ARD_8-11_5V-24V.2; no longer J_ARD.5
- net N$28: now also EN_M1_ENC_PHZ.2, J5/J7.9; no longer J_ARD.6
- net N$30: now also J5/J7.10; no longer J_ARD.7
- net OUT_3V3_SCI_TX: now also U6.1A1
- net OUT_5V_M1_CCW_INIB: now also J_ARD.7
- net OUT_5V_M1_CW_INIB: now also J_ARD.6
- net OUT_5V_M2_CCW_INIB: now also J_ARD.9
- net OUT_5V_M2_CW_INIB: now also J_ARD.8
- net OUT_5V_TX: now also J_ARD.5, U6.2A4; no longer J_ARD.4

Commit message: 13/03/2021
Parts:
- removed GPO1_24V, GPO2_24V, GPO3_24V, GPO4_24V, M1_BKW_INIB, M1_FWD_INIB, M1_RUN, M2_BKW_INIB, M2_BRAKE, M2_FWD_INIB, M2_RUN, MZ_EN: AGQ20003, SCARA:AGQ20003
- added IC12, IC13, IC14: LM324N, SCARA:LM324N
- added JI_ARD: 61202021621, SCARA:61202021621
- added MOTZ_2: 61201021621, SCARA:61201021621
- added R20, R21, R22, R23, R24: 4k7, rcl:R-EU_0207/10
- added R25: 47k, SCARA:R-EU_0204/7
- added R26: VS_ARD_ADJ, SCARA:64WR5KLF
- R1, R10, R11, R12, R13, R2, R3, R4, R6, R7, R8, R9: device SCARA:R-EU_0204/7 -> rcl:R-EU_0207/10
- renumbered MOTZ to MOTZ_1
Connections:
- removed net N$17: M1_BKW_INIB.1, U$2.1, U1.OUT2
- removed net N$19: M1_RUN.1, U$3.1, U1.OUT3
- removed net N$21: M2_FWD_INIB.1, U$4.1, U1.OUT4
- removed net N$23: M2_BKW_INIB.1, U$5.1, U1.OUT5
- removed net N$25: M2_RUN.1, U$6.1, U1.OUT6
- removed net N$27: M2_BRAKE.1, U$7.1, U1.OUT7
- removed net N$29: MZ_EN.1, U$8.1, U2.OUT1
- removed net N$31: GPO1_24V.1, U$9.1, U2.OUT2
- removed net N$33: GPO2_24V.1, U$10.1, U2.OUT3
- removed net N$35: GPO3_24V.1, U$11.1, U2.OUT4
- removed net N$37: GPO4_24V.1, U$12.1, U2.OUT5
- removed net OUT1_NC: GPO1_24V.2
- removed net OUT1_NO: GPO1_24V.4
- removed net OUT2_NC: GPO2_24V.2
- removed net OUT2_NO: GPO2_24V.4
- removed net OUT3_NC: GPO3_24V.2
- removed net OUT3_NO: GPO3_24V.4
- removed net OUT4_NC: GPO4_24V.2
- removed net OUT4_NO: GPO4_24V.4
- new net GPO1_24V: R22.1, U$10.1, U2.OUT3
- new net GPO2_24V: R23.1, U$11.1, U2.OUT4
- new net GPO3_24V: R24.1, U$12.1, U2.OUT5
- new net IN_30V_GPI1: IC12B.+IN, JI_ARD.2
- new net IN_30V_GPI10: IC14C.+IN, JI_ARD.20
- new net IN_30V_GPI2: IC12C.+IN, JI_ARD.4
- new net IN_30V_GPI3: IC12D.+IN, JI_ARD.6
- new net IN_30V_GPI4: IC13A.+IN, JI_ARD.8
- new net IN_30V_GPI5: IC13B.+IN, JI_ARD.10
- new net IN_30V_GPI6: IC13C.+IN, JI_ARD.12
- new net IN_30V_GPI7: IC13D.+IN, JI_ARD.14
- new net IN_30V_GPI8: IC14A.+IN, JI_ARD.16
- new net IN_30V_GPI9: IC14B.+IN, JI_ARD.18
- new net OUT_MZ_HOMING: MOTZ_2.1, R21.1, U$9.1, U2.OUT2
- new net VS_IN_ARD: IC12A.-IN, IC12A.OUT, IC12B.-IN, IC12C.-IN, IC12D.-IN, IC13A.-IN, IC13B.-IN, IC13C.-IN, IC13D.-IN, IC14A.-IN, IC14B.-IN, IC14C.-IN
- net +24V: now also R20.2, R21.2, R22.2, R23.2, R24.2, R25.2; no longer GPO1_24V.3, GPO2_24V.3, GPO3_24V.3, GPO4_24V.3, M1_BKW_INIB.3, M1_FWD_INIB.3, M1_RUN.3, M2_BKW_INIB.3, M2_BRAKE.3, M2_FWD_INIB.3, M2_RUN.3, MZ_EN.3
- net +5V: now also IC12P.V+, IC13P.V+, IC14P.V+; no longer GPO1_24V.8, GPO2_24V.8, GPO3_24V.8, GPO4_24V.8, M1_BKW_INIB.8, M1_FWD_INIB.8, M1_RUN.8, M2_BKW_INIB.8, M2_BRAKE.8, M2_FWD_INIB.8, M2_RUN.8, MZ_EN.8
- net GND: now also IC12P.V-, IC13P.V-, IC14P.V-, JI_ARD.1, JI_ARD.11, JI_ARD.13, JI_ARD.15, JI_ARD.17, JI_ARD.19, JI_ARD.3, JI_ARD.5, JI_ARD.7, JI_ARD.9, R26.1
- net IN_5V_GPI10_0V-30V: now also IC14C.OUT
- net IN_5V_GPI1_0V-30V: now also IC12B.OUT
- net IN_5V_GPI2_0V-30V: now also IC12C.OUT
- net IN_5V_GPI3_0V-30V: now also IC12D.OUT
- net IN_5V_GPI4_0V-30V: now also IC13A.OUT
- net IN_5V_GPI5_0V-30V: now also IC13B.OUT
- net IN_5V_GPI6_0V-30V: now also IC13C.OUT
- net IN_5V_GPI7_0V-30V: now also IC13D.OUT
- net IN_5V_GPI8_0V-30V: now also IC14A.OUT
- net IN_5V_GPI9_0V-30V: now also IC14B.OUT
- net N$15: now also IC12A.+IN, R25.1, R26.3; no longer M1_FWD_INIB.1, U$1.1, U1.OUT1
- net OUT_M1_BKW_INIB: now also U$2.1, U1.OUT2; no longer M1_BKW_INIB.2
- net OUT_M1_FWD_INIB: now also U$1.1, U1.OUT1; no longer M1_FWD_INIB.2
- net OUT_M1_RUN: now also U$3.1, U1.OUT3; no longer M1_RUN.4
- net OUT_M2_BKW_INIB: now also U$5.1, U1.OUT5; no longer M2_BKW_INIB.2
- net OUT_M2_BRAKE: now also U$7.1, U1.OUT7; no longer M2_BRAKE.4
- net OUT_M2_FWD_INIB: now also U$4.1, U1.OUT4; no longer M2_FWD_INIB.2
- net OUT_M2_RUN: now also U$6.1, U1.OUT6; no longer M2_RUN.4
- net OUT_MZ_EN: now also R20.1, U$8.1, U2.OUT1; no longer MZ_EN.4
