File: Tesi/comando 24V.sch (EAGLE design)
At the start: 87 parts, among them IC1 LM324N, IC10 LM324N, IC11 LM324N, IC12 LM324N, IC13 LM324N, IC14 LM324N, IC2 LM324N, IC3 LM324N, IC4 LM324N, IC5 LM324N, IC6 LM324N, IC7 LM324N, IC8 LM324N, IC9 LM324N, J1/J3 61202021621, J10 SBH11-PBPC-D25-ST-BK, J4/J2 61202021621, J5/J7 61202021621, J8/J6 61202021621, J9 SBH11-PBPC-D25-ST-BK, U1 ULN2003A, U2 ULN2003A, U3 TMP37FT9Z, U4 SN74LS244N, U5 SN74LS244N, U6 SN74LS244N

Commit message: fine giornata
Connections:
- removed net N$100: J_ARD.43
- removed net N$101: J_ARD.44
- removed net N$102: J_ARD.45
- removed net N$103: J_ARD.46
- removed net N$104: J_ARD.47
- removed net N$105: J_ARD.48
- removed net N$106: J_ARD.49
- removed net N$107: J_ARD.50
- removed net N$95: J_ARD.40
- removed net N$98: J_ARD.41
- removed net N$99: J_ARD.42
Changed lines of the file:
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@@
 <part name="GND5" library="supply1" library_urn="urn:adsk.eagle:library:371" deviceset="GND" device=""/>
 <part name="JI_ARD" library="SCARA" deviceset="61202021621" device=""/>
+<part name="FRAME10" library="frames" library_urn="urn:adsk.eagle:library:229" deviceset="A4L-LOC" device=""/>
 </parts>
 <sheets>
@@
 <segment>
 <pinref part="MOT2" gate="A" pin="34"/>
-<wire x1="157.48" y1="80.01" x2="128.27" y2="80.01" width="0.1524" layer="91"/>
-<label x="128.27" y="80.01" size="1.6764" layer="95" rot="R180" xref="yes"/>
+<wire x1="157.48" y1="80.01" x2="124.46" y2="80.01" width="0.1524" layer="91"/>
+<label x="124.46" y="80.01" size="1.6764" layer="95" rot="R180" xref="yes"/>
 </segment>
 <segment>
 <pinref part="MOT2" gate="A" pin="36"/>
-<wire x1="157.48" y1="74.93" x2="128.27" y2="74.93" width="0.1524" layer="91"/>
-<label x="128.27" y="74.93" size="1.6764" layer="95" rot="R180" xref="yes"/>
+<wire x1="157.48" y1="74.93" x2="124.46" y2="74.93" width="0.1524" layer="91"/>
+<label x="124.46" y="74.93" size="1.6764" layer="95" rot="R180" xref="yes"/>
 </segment>
 <segment>
 <pinref part="MOT2" gate="A" pin="38"/>
-<wire x1="157.48" y1="69.85" x2="132.08" y2="69.85" width="0.1524" layer="91"/>
-<label x="132.08" y="69.85" size="1.6764" layer="95" rot="R180" xref="yes"/>
+<wire x1="157.48" y1="69.85" x2="124.46" y2="69.85" width="0.1524" layer="91"/>
+<label x="124.46" y="69.85" size="1.6764" layer="95" rot="R180" xref="yes"/>
 </segment>
 <segment>
@@
 <segment>
 <pinref part="MOT1" gate="A" pin="34"/>
-<wire x1="240.03" y1="80.01" x2="210.82" y2="80.01" width="0.1524" layer="91"/>
-<label x="210.82" y="80.01" size="1.6764" layer="95" rot="R180" xref="yes"/>
+<wire x1="240.03" y1="80.01" x2="207.01" y2="80.01" width="0.1524" layer="91"/>
+<label x="207.01" y="80.01" size="1.6764" layer="95" rot="R180" xref="yes"/>
 </segment>
 <segment>
 <pinref part="MOT1" gate="A" pin="36"/>
-<wire x1="240.03" y1="74.93" x2="210.82" y2="74.93" width="0.1524" layer="91"/>
-<label x="210.82" y="74.93" size="1.6764" layer="95" rot="R180" xref="yes"/>
+<wire x1="240.03" y1="74.93" x2="207.01" y2="74.93" width="0.1524" layer="91"/>
+<label x="207.01" y="74.93" size="1.6764" layer="95" rot="R180" xref="yes"/>
 </segment>
 <segment>
 <pinref part="MOT1" gate="A" pin="38"/>
-<wire x1="240.03" y1="69.85" x2="214.63" y2="69.85" width="0.1524" layer="91"/>
-<label x="214.63" y="69.85" size="1.6764" layer="95" rot="R180" xref="yes"/>
+<wire x1="240.03" y1="69.85" x2="207.01" y2="69.85" width="0.1524" layer="91"/>
+<label x="207.01" y="69.85" size="1.6764" layer="95" rot="R180" xref="yes"/>
 </segment>
 <segment>
@@
 <segment>
 <pinref part="J_ARD" gate="A" pin="4"/>
-<wire x1="156.21" y1="153.67" x2="138.43" y2="153.67" width="0.1524" layer="91"/>
-<label x="138.43" y="153.67" size="1.6764" layer="95" rot="R180" xref="yes"/>
+<wire x1="156.21" y1="153.67" x2="133.35" y2="153.67" width="0.1524" layer="91"/>
+<label x="133.35" y="153.67" size="1.6764" layer="95" rot="R180" xref="yes"/>
 </segment>
 </net>
@@
 <segment>
 <pinref part="J_ARD" gate="A" pin="28"/>
-<wire x1="156.21" y1="92.71" x2="124.46" y2="92.71" width="0.1524" layer="91"/>
-<label x="124.46" y="92.71" size="1.6764" layer="95" rot="R180" xref="yes"/>
+<wire x1="156.21" y1="92.71" x2="123.19" y2="92.71" width="0.1524" layer="91"/>
+<label x="123.19" y="92.71" size="1.6764" layer="95" rot="R180" xref="yes"/>
 </segment>
 </net>
@@
 <segment>
 <pinref part="J_ARD" gate="A" pin="30"/>
-<wire x1="156.21" y1="87.63" x2="128.27" y2="87.63" width="0.1524" layer="91"/>
-<label x="128.27" y="87.63" size="1.6764" layer="95" rot="R180" xref="yes"/>
+<wire x1="156.21" y1="87.63" x2="123.19" y2="87.63" width="0.1524" layer="91"/>
+<label x="123.19" y="87.63" size="1.6764" layer="95" rot="R180" xref="yes"/>
 </segment>
 </net>
@@
 <segment>
 <pinref part="J_ARD" gate="A" pin="32"/>
-<wire x1="156.21" y1="82.55" x2="128.27" y2="82.55" width="0.1524" layer="91"/>
-<label x="128.27" y="82.55" size="1.6764" layer="95" rot="R180" xref="yes"/>
+<wire x1="156.21" y1="82.55" x2="123.19" y2="82.55" width="0.1524" layer="91"/>
+<label x="123.19" y="82.55" size="1.6764" layer="95" rot="R180" xref="yes"/>
 </segment>
 </net>
@@
 <segment>
 <pinref part="J_ARD" gate="A" pin="34"/>
-<wire x1="156.21" y1="77.47" x2="128.27" y2="77.47" width="0.1524" layer="91"/>
-<label x="128.27" y="77.47" size="1.6764" layer="95" rot="R180" xref="yes"/>
+<wire x1="156.21" y1="77.47" x2="123.19" y2="77.47" width="0.1524" layer="91"/>
+<label x="123.19" y="77.47" size="1.6764" layer="95" rot="R180" xref="yes"/>
 </segment>
 </net>
@@
 <segment>
 <pinref part="J_ARD" gate="A" pin="36"/>
-<wire x1="156.21" y1="72.39" x2="127" y2="72.39" width="0.1524" layer="91"/>
-<label x="127" y="72.39" size="1.6764" layer="95" rot="R180" xref="yes"/>
+<wire x1="156.21" y1="72.39" x2="123.19" y2="72.39" width="0.1524" layer="91"/>
+<label x="123.19" y="72.39" size="1.6764" layer="95" rot="R180" xref="yes"/>
 </segment>
 </net>
@@
 </segment>
 </net>
-<net name="N$95" class="0">
-<segment>
-<pinref part="J_ARD" gate="A" pin="40"/>
-<wire x1="156.21" y1="62.23" x2="154.94" y2="62.23" width="0.1524" layer="91"/>
-<label x="154.94" y="62.23" size="1.6764" layer="95" rot="R180" xref="yes"/>
-</segment>
-</net>
-<net name="N$98" class="0">
-<segment>
-<pinref part="J_ARD" gate="A" pin="41"/>
-<wire x1="156.21" y1="59.69" x2="154.94" y2="59.69" width="0.1524" layer="91"/>
-<label x="154.94" y="59.69" size="1.6764" layer="95" rot="R180" xref="yes"/>
-</segment>
-</net>
-<net name="N$99" class="0">
-<segment>
-<pinref part="J_ARD" gate="A" pin="42"/>
-<wire x1="156.21" y1="57.15" x2="154.94" y2="57.15" width="0.1524" layer="91"/>
-<label x="154.94" y="57.15" size="1.6764" layer="95" rot="R180" xref="yes"/>
-</segment>
-</net>
-<net name="N$100" class="0">
-<segment>
-<pinref part="J_ARD" gate="A" pin="43"/>
-<wire x1="156.21" y1="54.61" x2="154.94" y2="54.61" width="0.1524" layer="91"/>
-<label x="154.94" y="54.61" size="1.6764" layer="95" rot="R180" xref="yes"/>
-</segment>
-</net>
-<net name="N$101" class="0">
-<segment>
-<pinref part="J_ARD" gate="A" pin="44"/>
-<wire x1="156.21" y1="52.07" x2="154.94" y2="52.07" width="0.1524" layer="91"/>
-<label x="154.94" y="52.07" size="1.6764" layer="95" rot="R180" xref="yes"/>
-</segment>
-</net>
-<net name="N$102" class="0">
-<segment>
-<pinref part="J_ARD" gate="A" pin="45"/>
-<wire x1="156.21" y1="49.53" x2="154.94" y2="49.53" width="0.1524" layer="91"/>
-<label x="154.94" y="49.53" size="1.6764" layer="95" rot="R180" xref="yes"/>
-</segment>
-</net>
-<net name="N$103" class="0">
-<segment>
-<pinref part="J_ARD" gate="A" pin="46"/>
-<wire x1="156.21" y1="46.99" x2="154.94" y2="46.99" width="0.1524" layer="91"/>
-<label x="154.94" y="46.99" size="1.6764" layer="95" rot="R180" xref="yes"/>
-</segment>
-</net>
-<net name="N$104" class="0">
-<segment>
-<pinref part="J_ARD" gate="A" pin="47"/>
-<wire x1="156.21" y1="44.45" x2="154.94" y2="44.45" width="0.1524" layer="91"/>
-<label x="154.94" y="44.45" size="1.6764" layer="95" rot="R180" xref="yes"/>
-</segment>
-</net>
-<net name="N$105" class="0">
-<segment>
-<pinref part="J_ARD" gate="A" pin="48"/>
-<wire x1="156.21" y1="41.91" x2="154.94" y2="41.91" width="0.1524" layer="91"/>
-<label x="154.94" y="41.91" size="1.6764" layer="95" rot="R180" xref="yes"/>
-</segment>
-</net>
-<net name="N$106" class="0">
-<segment>
-<pinref part="J_ARD" gate="A" pin="49"/>
-<wire x1="156.21" y1="39.37" x2="154.94" y2="39.37" width="0.1524" layer="91"/>
-<label x="154.94" y="39.37" size="1.6764" layer="95" rot="R180" xref="yes"/>
-</segment>
-</net>
-<net name="N$107" class="0">
-<segment>
-<pinref part="J_ARD" gate="A" pin="50"/>
-<wire x1="156.21" y1="36.83" x2="154.94" y2="36.83" width="0.1524" layer="91"/>
-<label x="154.94" y="36.83" size="1.6764" layer="95" rot="R180" xref="yes"/>
-</segment>
-</net>
 <net name="OUT_5V_TX" class="0">
 <segment>
@@
 </nets>
 </sheet>
+<sheet>
+<plain>
+</plain>
+<instances>
+<instance part="FRAME10" gate="G$1" x="0" y="0" smashed="yes">
+<attribute name="DRAWING_NAME" x="217.17" y="15.24" size="2.54" layer="94"/>
+<attribute name="LAST_DATE_TIME" x="217.17" y="10.16" size="2.286" layer="94"/>
+<attribute name="SHEET" x="230.505" y="5.08" size="2.54" layer="94"/>
+</instance>
+</instances>
+<busses>
+</busses>
+<nets>
+</nets>
+</sheet>

Commit message: fine schematico
Parts:
- added EN_GPO_H: STRIP_3, SCARA:STRIP_3
- added IC15, IC16, IC17: LM324N, SCARA:LM324N
- added JI_ARD1, J_GPO/I2C_H1: 61202021621, SCARA:61202021621
- added R27: 47k, rcl:R-EU_0207/10
- added R28: VS_EDGE_ADJ, SCARA:64WR5KLF
- added R29: 2K, rcl:R-EU_0207/10
- added U$15: LED_ON, SCARA:LED_TONDO
- added U7: SN74LS244N, SCARA:SN74LS244N
- R14, R16, R18, R25: device SCARA:R-EU_0204/7 -> rcl:R-EU_0207/10
Connections:
- removed net IN_3V3_24V_ALARM: IC2B.OUT
- removed net IN_3V3_TENS_ALARM: J9.15
- removed net IN_5V_GPI11_0V-30V: J_ARD.37
- removed net N$36: J4/J2.5
- removed net N$38: J4/J2.7
- removed net N$40: J4/J2.9
- removed net N$41: J4/J2.11
- removed net N$54: J4/J2.4
- removed net N$55: J4/J2.6
- removed net N$56: J4/J2.18
- removed net N$62: J5/J7.19
- removed net N$70: J8/J6.16
- removed net N$71: J8/J6.18
- removed net N$84: J10.10
- removed net N$85: J10.12
- removed net N$89: J10.20
- removed net N$92: J10.25
- removed net N$93: J10.27
- removed net N$94: J10.28
- removed net N$97: J10.39
- new net I/O_3V3_GPIO1: J10.39, J_GPO/I2C_H1.20
- new net I/O_3V3_I2C_SCL: J10.8, J_GPO/I2C_H1.16
- new net I/O_3V3_I2C_SDA: J10.9, J_GPO/I2C_H1.18
- new net IN_30V_EDGE1: IC15B.+IN, JI_ARD1.2
- new net IN_30V_EDGE10: IC17C.+IN, JI_ARD1.20
- new net IN_30V_EDGE2: IC15C.+IN, JI_ARD1.4
- new net IN_30V_EDGE3: IC15D.+IN, JI_ARD1.6
- new net IN_30V_EDGE4: IC16A.+IN, JI_ARD1.8
- new net IN_30V_EDGE5: IC16B.+IN, JI_ARD1.10
- new net IN_30V_EDGE6: IC16C.+IN, JI_ARD1.12
- new net IN_30V_EDGE7: IC16D.+IN, JI_ARD1.14
- new net IN_30V_EDGE8: IC17A.+IN, JI_ARD1.16
- new net IN_30V_EDGE9: IC17B.+IN, JI_ARD1.18
- new net IN_3V3_EDGE1: IC15B.OUT, J4/J2.5
- new net IN_3V3_EDGE10: IC17C.OUT, J10.19
- new net IN_3V3_EDGE2: IC15C.OUT, J4/J2.9
- new net IN_3V3_EDGE3: IC15D.OUT, J4/J2.11
- new net IN_3V3_EDGE4: IC16A.OUT, J9.22
- new net IN_3V3_EDGE5: IC16B.OUT, J9.23
- new net IN_3V3_EDGE6: IC16C.OUT, J9.24
- new net IN_3V3_EDGE7: IC16D.OUT, J9.26
- new net IN_3V3_EDGE8: IC17A.OUT, J9.27
- new net IN_3V3_EDGE9: IC17B.OUT, J9.28
- new net N$17: IC15A.+IN, R27.1, R28.3
- new net N$19: EN_GPO_H.2, U7.!1G, U7.!G/2G
- new net N$21: R29.1, U$15.2
- new net OUT_3V3_GPO1_H: J9.10, U7.1A1
- new net OUT_3V3_GPO2_H: J9.11, U7.1A2
- new net OUT_3V3_GPO3_H: J9.14, U7.1A3
- new net OUT_3V3_GPO4_H: J9.17, U7.1A4
- new net OUT_3V3_GPO5_H: J9.18, U7.2A4
- new net OUT_3V3_GPO6_H: J10.34, U7.2A3
- new net OUT_3V3_GPO7_H: J9.20, U7.2A2
- new net OUT_5V_GPO1_H: J_GPO/I2C_H1.2, U7.1Y1
- new net OUT_5V_GPO2_H: J_GPO/I2C_H1.4, U7.1Y2
- new net OUT_5V_GPO3_H: J_GPO/I2C_H1.6, U7.1Y3
- new net OUT_5V_GPO4_H: J_GPO/I2C_H1.8, U7.1Y4
- new net OUT_5V_GPO5_H: J_GPO/I2C_H1.10, U7.2Y4
- new net OUT_5V_GPO6_H: J_GPO/I2C_H1.12, U7.2Y3
- new net OUT_5V_GPO7_H: J_GPO/I2C_H1.14, U7.2Y2
- new net VS_IN_EDGE: IC15A.-IN, IC15A.OUT, IC15B.-IN, IC15C.-IN, IC15D.-IN, IC16A.-IN, IC16B.-IN, IC16C.-IN, IC16D.-IN, IC17A.-IN, IC17B.-IN, IC17C.-IN
- net +24V: now also R27.2, R29.2; no longer IC2B.+IN
- net +3V3: now also IC15P.V+, IC16P.V+, IC17P.V+; no longer IC2B.-IN
- net +5V: now also EN_GPO_H.1, U7.VCC
- net GND: now also EN_GPO_H.3, IC15P.V-, IC16P.V-, IC17P.V-, JI_ARD1.1, JI_ARD1.11, JI_ARD1.13, JI_ARD1.15, JI_ARD1.17, JI_ARD1.19, JI_ARD1.3, JI_ARD1.5, JI_ARD1.7, JI_ARD1.9, J_GPO/I2C_H1.1, J_GPO/I2C_H1.11, J_GPO/I2C_H1.13, J_GPO/I2C_H1.15, J_GPO/I2C_H1.17, J_GPO/I2C_H1.19, J_GPO/I2C_H1.3, J_GPO/I2C_H1.5, J_GPO/I2C_H1.7, J_GPO/I2C_H1.9, R28.1, U$15.1, U7.GND
- net IN_3V3_220V_ALARM: now also J9.15
- net IN_3V3_M1_ENC_PHA: now also J1/J3.13; no longer J5/J7.13
- net OUT_3V3_M2_CW: now also J8/J6.7; no longer J9.6

Commit message: fine schematico parte 2
Parts:
- added J1, J2, J3, J4, J5, J6: 61201021621, SCARA:61201021621
Connections:
- removed net IN_3V3_M1_BKIR: MOT1.11
- removed net IN_3V3_M1_GPO1: MOT1.12
- removed net IN_3V3_M1_GPO2: MOT1.40
- removed net IN_3V3_M1_INP: MOT1.39
- removed net IN_3V3_M1_PHZ: MOT1.19
- removed net IN_3V3_M2_BKIR: MOT2.11
- removed net IN_3V3_M2_GPO1: MOT2.12
- removed net IN_3V3_M2_GPO2: MOT2.40
- removed net IN_3V3_M2_INP: MOT2.39
- removed net IN_3V3_M2_PHZ: MOT2.19
- removed net M1_BAT: MOT1.42
- removed net M1_BATCOM: MOT1.43
- removed net M2_BAT: MOT2.42
- removed net M2_BATCOM: MOT2.43
- removed net N$45: MOT1.13, MOT2.13
- removed net N$46: MOT1.14, MOT2.14
- removed net N$47: MOT1.15, MOT2.15
- removed net N$48: MOT1.16, MOT2.16
- removed net N$49: MOT1.17, MOT2.17
- removed net N$50: MOT1.18, MOT2.18
- removed net N$52: MOT1.20, MOT2.20
- removed net N$87: MOT1.50, MOT2.50
- removed net OUT_24V_M1_CCW: MOT1.2
- removed net OUT_24V_M1_CW: MOT1.1
- removed net OUT_24V_M1_DFSEL: MOT1.26
- removed net OUT_24V_M1_ECRST: MOT1.30
- removed net OUT_24V_M1_GESEL: MOT1.28
- removed net OUT_24V_M1_GSEL: MOT1.27
- removed net OUT_24V_M1_IPG: MOT1.33
- removed net OUT_24V_M1_RESET: MOT1.31
- removed net OUT_24V_M1_TVSEL: MOT1.32
- removed net OUT_24V_M2_CCW: MOT2.2
- removed net OUT_24V_M2_CW: MOT2.1
- removed net OUT_24V_M2_DFSEL: MOT2.26
- removed net OUT_24V_M2_ECRST: MOT2.30
- removed net OUT_24V_M2_GESEL: MOT2.28
- removed net OUT_24V_M2_GSEL: MOT2.27
- removed net OUT_24V_M2_IPG: MOT2.33
- removed net OUT_24V_M2_RESET: MOT2.31
- removed net OUT_24V_M2_TVSEL: MOT2.32
- removed net OUT_5V_M1_CCWLD: MOT1.46
- removed net OUT_5V_M1_CWLD: MOT1.44
- removed net OUT_5V_M2_CCWLD: MOT2.46
- removed net OUT_5V_M2_CWLD: MOT2.44
- new net I/O_M1_1: J4.1, MOT1.1
- new net I/O_M1_11: J4.3, MOT1.11
- new net I/O_M1_12: J4.4, MOT1.12
- new net I/O_M1_13: J4.5, MOT1.13
- new net I/O_M1_14: J4.6, MOT1.14
- new net I/O_M1_15: J4.7, MOT1.15
- new net I/O_M1_16: J4.8, MOT1.16
- new net I/O_M1_17: J4.9, MOT1.17
- new net I/O_M1_18: J4.10, MOT1.18
- new net I/O_M1_19: J5.1, MOT1.19
- new net I/O_M1_2: J4.2, MOT1.2
- new net I/O_M1_20: J5.2, MOT1.20
- new net I/O_M1_26: J5.3, MOT1.26
- new net I/O_M1_27: J5.4, MOT1.27
- new net I/O_M1_28: J5.5, MOT1.28
- new net I/O_M1_30: J5.6, MOT1.30
- new net I/O_M1_31: J5.7, MOT1.31
- new net I/O_M1_32: J5.8, MOT1.32
- new net I/O_M1_33: J5.9, MOT1.33
- new net I/O_M1_39: J5.10, MOT1.39
- new net I/O_M1_40: J6.1, MOT1.40
- new net I/O_M1_42: J6.2, MOT1.42
- new net I/O_M1_43: J6.3, MOT1.43
- new net I/O_M1_44: J6.4, MOT1.44
- new net I/O_M1_46: J6.5, MOT1.46
- new net I/O_M1_50: J6.6, MOT1.50
- new net I/O_M2_1: J1.1, MOT2.1
- new net I/O_M2_11: J1.3, MOT2.11
- new net I/O_M2_12: J1.4, MOT2.12
- new net I/O_M2_13: J1.5, MOT2.13
- new net I/O_M2_14: J1.6, MOT2.14
- new net I/O_M2_15: J1.7, MOT2.15
- new net I/O_M2_16: J1.8, MOT2.16
- new net I/O_M2_17: J1.9, MOT2.17
- new net I/O_M2_18: J1.10, MOT2.18
- new net I/O_M2_19: J2.1, MOT2.19
- new net I/O_M2_2: J1.2, MOT2.2
- new net I/O_M2_20: J2.2, MOT2.20
- new net I/O_M2_26: J2.3, MOT2.26
- new net I/O_M2_27: J2.4, MOT2.27
- new net I/O_M2_28: J2.5, MOT2.28
- new net I/O_M2_30: J2.6, MOT2.30
- new net I/O_M2_31: J2.7, MOT2.31
- new net I/O_M2_32: J2.8, MOT2.32
- new net I/O_M2_33: J2.9, MOT2.33
- new net I/O_M2_39: J2.10, MOT2.39
- new net I/O_M2_40: J3.1, MOT2.40
- new net I/O_M2_42: J3.2, MOT2.42
- new net I/O_M2_43: J3.3, MOT2.43
- new net I/O_M2_44: J3.4, MOT2.44
- new net I/O_M2_46: J3.5, MOT2.46
- new net I/O_M2_50: J3.6, MOT2.50
