File: Tesi/comando 24V.sch (EAGLE design)
At the start: 104 parts, among them IC1 LM324N, IC10 LM324N, IC11 LM324N, IC12 LM324N, IC13 LM324N, IC14 LM324N, IC15 LM324N, IC16 LM324N, IC17 LM324N, IC2 LM324N, IC3 LM324N, IC4 LM324N, IC5 LM324N, IC6 LM324N, IC7 LM324N, IC8 LM324N, IC9 LM324N, J1 61201021621, J1/J3 61202021621, J10 SBH11-PBPC-D25-ST-BK, J2 61201021621, J3 61201021621, J4 61201021621, J4/J2 61202021621, J5 61201021621, J5/J7 61202021621, J6 61201021621, J8/J6 61202021621, J9 SBH11-PBPC-D25-ST-BK, U1 ULN2003A, U2 ULN2003A, U3 TMP37FT9Z, U4 SN74LS244N, U5 SN74LS244N, U6 SN74LS244N, U7 SN74LS244N

Commit message: 16/03/2021
Connections:
- net +3V3: no longer IC15P.V+, IC16P.V+, IC17P.V+, IC1P.V+, IC2P.V+, IC3P.V+
- net +5V: now also IC15P.V+, IC16P.V+, IC17P.V+, IC1P.V+, IC2P.V+, IC3P.V+
Other:
- moved on the sheet: R1, R10, R11, R12, R13, R2, R20, R21, R22, R23, R24, R3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

Commit message: 20/03/2021 mattina
Parts:
- removed IC10, IC6, IC8: LM324N, SCARA:LM324N
- removed IC4, IC9: LM324N, linear:LM324N
- added EL_VALV: CON_2F, SCARA:CON_2F
- added J7: 61201021621, SCARA:61201021621
- added J8: 61202021621, SCARA:61202021621
- added U8: H11L1M, SCARA:H11L1M
- renumbered JI_ARD1 to JI_TEXAS
Connections:
- removed net 220V_PRB: PT1.2
- removed net GPO1_24V: R22.1, U$10.1, U2.OUT3
- removed net GPO2_24V: R23.1, U$11.1, U2.OUT4
- removed net GPO3_24V: R24.1, U$12.1, U2.OUT5
- removed net OUT_5V_GPO3_24V: J_ARD.19, U2.IN5
- new net GND_220V: PT1.1, U$13.2, U$14.-, U8.CATHODE
- new net N$23: PT1.3, R5.1
- new net OUT_24V_ELVALV: EL_VALV.1, R22.1, U$10.1, U2.OUT3
- new net OUT_24V_GPO1: J7.1, R23.1, U$11.1, U2.OUT4
- new net OUT_24V_GPO2: J7.3, R24.1, U$12.1, U2.OUT5
- new net OUT_5V_ELVALV_24V: J_ARD.17, U2.IN3
- net +24V: now also EL_VALV.2, U1.COMMON, U2.COMMON
- net +3V3: now also IC1B.-IN, IC1D.-IN, U8.VCC; no longer IC10B.-IN, IC2A.-IN, IC4D.-IN
- net +5V: no longer U1.COMMON, U2.COMMON
- net 220V_PROBE: now also PT1.2, U8.ANODE; no longer IC2A.+IN, PT1.3, R5.1
- net GND: now also J7.2, J7.4, J8.1, J8.11, J8.13, J8.15, J8.17, J8.19, J8.3, J8.5, J8.7, J8.9, U8.GND; no longer PT1.1, U$13.2, U$14.-
- net IN_24V_HOMING_SENS_M2: now also IC1B.+IN; no longer IC10B.+IN
- net IN_24V_MZ_ENC_CW: now also IC1D.+IN; no longer IC4D.+IN
- net IN_3V3_220V_ALARM: now also U8.VO; no longer IC2A.OUT
- net IN_3V3_HOMING_SENS_M2: now also IC1B.OUT; no longer IC10B.OUT
- net IN_3V3_MZ_ENC_CW: now also IC1D.OUT; no longer IC4D.OUT
- net IN_3V3_TEMP_ALARM: now also IC1C.OUT; no longer IC8D.OUT
- net N$14: now also IC2B.+IN; no longer IC9C.+IN
- net N$39: now also IC5D.+IN; no longer IC6D.+IN
- net OUT_24V-5V_GPO10: now also J8.14
- net OUT_24V-5V_GPO4: now also J8.2
- net OUT_24V-5V_GPO5: now also J8.4
- net OUT_24V-5V_GPO6: now also J8.6
- net OUT_24V-5V_GPO7: now also J8.8
- net OUT_24V-5V_GPO8: now also J8.10
- net OUT_24V-5V_GPO9: now also J8.12
- net OUT_5V_GPO1_24V: now also J_ARD.18, U2.IN4; no longer J_ARD.17, U2.IN3
- net OUT_5V_GPO2_24V: now also J_ARD.19, U2.IN5; no longer J_ARD.18, U2.IN4
- net TEMP: now also IC1C.+IN; no longer IC8D.+IN
- net VS_3V3: now also IC5D.-IN, IC5D.OUT; no longer IC6D.-IN, IC6D.OUT
- net VS_TEMP: now also IC1C.-IN, IC2B.-IN, IC2B.OUT; no longer IC8D.-IN, IC9C.-IN, IC9C.OUT
Other:
- moved on the sheet: 24V_SUP, AC_SUP, IC7A, IC7B, IC7C, J1, J2, J3, J4, J5, J6, MOTZ_1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

Commit message: 23/03/2021 placing
Parts:
- added C1: UMF1V010MDD1TP, SCARA:UMF1V010MDD1TP
Connections:
- net +24V: now also C1.1
- net GND: now also C1.2
Changed lines of the file:
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@@
 <part name="J8" library="SCARA" deviceset="61202021621" device=""/>
 <part name="U8" library="SCARA" deviceset="H11L1M" device=""/>
+<part name="C1" library="SCARA" deviceset="UMF1V010MDD1TP" device=""/>
 </parts>
 <sheets>
@@
 <attribute name="VALUE" x="109.982" y="107.95" size="1.778" layer="96" rot="R90"/>
 </instance>
+<instance part="C1" gate="A" x="128.27" y="113.03" smashed="yes" rot="R270">
+<attribute name="NAME" x="131.6228" y="112.0394" size="1.778" layer="95" ratio="10" rot="SR270"/>
+</instance>
 </instances>
 <busses>
@@
 <label x="106.68" y="87.63" size="1.778" layer="95" rot="R180"/>
 </segment>
+<segment>
+<pinref part="C1" gate="A" pin="2"/>
+<wire x1="128.27" y1="105.41" x2="128.27" y2="102.87" width="0.1524" layer="91"/>
+<label x="128.27" y="102.87" size="1.778" layer="95" rot="R180"/>
+</segment>
 </net>
 <net name="220V_PROBE" class="0">
@@
 </segment>
 </net>
-<net name="AC_IN2" class="0">
+<net name="AC_IN2" class="1">
 <segment>
 <pinref part="U$14" gate="A" pin="AC2"/>
@@
 </segment>
 </net>
-<net name="AC_IN1" class="0">
+<net name="AC_IN1" class="1">
 <segment>
 <pinref part="U$14" gate="A" pin="AC1"/>
@@
 <wire x1="106.68" y1="116.84" x2="106.68" y2="118.11" width="0.1524" layer="91"/>
 <label x="106.68" y="118.11" size="1.778" layer="95"/>
+</segment>
+<segment>
+<pinref part="C1" gate="A" pin="1"/>
+<wire x1="128.27" y1="113.03" x2="128.27" y2="114.3" width="0.1524" layer="91"/>
+<wire x1="128.27" y1="114.3" x2="128.27" y2="115.57" width="0.1524" layer="91"/>
+<label x="128.27" y="115.57" size="1.778" layer="95"/>
 </segment>
 </net>
@@
 </busses>
 <nets>
-<net name="AC_IN1" class="0">
+<net name="AC_IN1" class="1">
 <segment>
 <pinref part="AC_SUP" gate="A" pin="1"/>
@@
 </segment>
 </net>
-<net name="AC_IN2" class="0">
+<net name="AC_IN2" class="1">
 <segment>
 <pinref part="AC_SUP" gate="A" pin="2"/>

Commit message: inizio routing
Connections:
- net IN_3V3_M1_ENC_PHA renamed IN_3V3_M1_ENC_PH_P
- net IN_3V3_M1_ENC_PHB renamed IN_3V3_M1_ENC_PH_N
- net IN_3V3_M2_ENC_PHA renamed IN_3V3_M2_ENC_PH_P
- net IN_3V3_M2_ENC_PHB renamed IN_3V3_M2_ENC_PH_N
- net IN_5V_M1_ENC_PHA renamed IN_5V_M1_ENC_PH_P
- net IN_5V_M1_ENC_PHB renamed IN_5V_M1_ENC_PH_N
- net IN_5V_M2_ENC_PHA renamed IN_5V_M2_ENC_PH_P
- net IN_5V_M2_ENC_PHB renamed IN_5V_M2_ENC_PH_N
- removed net N$39: IC5D.+IN, R18.1, R19.3
- new net N$25: IC12A.+IN, R26.2
- new net N$27: IC7D.+IN, R15.2
- new net N$29: IC5D.+IN, R19.2
- new net N$31: R18.1, R19.1
- new net N$32: IC2B.+IN, R17.2
- new net N$33: IC15A.+IN, R28.2
- net GND: now also R15.3, R17.3, R19.3, R26.3, R28.3; no longer R15.1, R17.1, R19.1, R26.1, R28.1
- net IN_30V_GPI1: now also IC12D.+IN; no longer IC12B.+IN
- net IN_30V_GPI3: now also IC12B.+IN; no longer IC12D.+IN
- net IN_5V_GPI3_0V-30V: now also IC13A.OUT; no longer IC12D.OUT
- net IN_5V_GPI4_0V-30V: now also IC13C.OUT; no longer IC13A.OUT
- net IN_5V_GPI5_0V-30V: now also IC13D.OUT; no longer IC13B.OUT
- net IN_5V_GPI6_0V-30V: now also IC12D.OUT; no longer IC13C.OUT
- net IN_5V_GPI7_0V-30V: now also IC13B.OUT; no longer IC13D.OUT
- net N$14: now also R17.1; no longer IC2B.+IN, R17.3
- net N$15: now also R26.1; no longer IC12A.+IN, R26.3
- net N$17: now also R28.1; no longer IC15A.+IN, R28.3
- net N$20: now also R15.1; no longer IC7D.+IN, R15.3
- net OUT_24V-5V_GPO4: now also IC11D.OUT; no longer IC11A.OUT
- net OUT_24V-5V_GPO5: now also IC11A.OUT; no longer IC11B.OUT
- net OUT_24V-5V_GPO6: now also IC11B.OUT; no longer IC11C.OUT
- net OUT_24V-5V_GPO7: now also IC11C.OUT; no longer IC11D.OUT
- net OUT_5V_M1_CCW_INIB: now also J_ARD.6; no longer J_ARD.7
- net OUT_5V_M1_CW_INIB: now also J_ARD.7; no longer J_ARD.6
- net OUT_5V_M2_CCW_INIB: now also J_ARD.8; no longer J_ARD.9
- net OUT_5V_M2_CW_INIB: now also J_ARD.9; no longer J_ARD.8
Other:
- moved on the sheet: IC7D, R15, R17, R19, R26, R28

Commit message: 28/03/2021
Parts:
- removed C1: UMF1V010MDD1TP, SCARA:UMF1V010MDD1TP
- removed IC2: LM324N, linear:LM324N
- removed IC3: LM324N, SCARA:LM324N
- added C2: QYX1H102JTP3TA, SCARA:QYX1H102JTP3TA
- added C3: UBY2A301MHL, SCARA:UBY2A301MHL
Connections:
- removed net IN_3V3_MZ_ENC_CCW: IC3A.OUT
- removed net IN_3V3_MZ_ENC_CW: IC1D.OUT
- removed net IN_3V3_MZ_ENC_PHZ: IC3B.OUT
- net +24V: now also C2.1, C3.1; no longer C1.1
- net +3V3: now also IC17D.-IN; no longer IC1D.-IN, IC3A.-IN, IC3B.-IN, IC3C.-IN
- net +5V: no longer IC2P.V+, IC3P.V+
- net GND: now also C2.2, C3.2; no longer C1.2, IC2P.V-, IC3P.V-
- net IN_24V_MZ_ALARM: now also IC17D.+IN; no longer IC3C.+IN
- net IN_24V_MZ_ENC_CCW: no longer IC3A.+IN
- net IN_24V_MZ_ENC_CW: no longer IC1D.+IN
- net IN_24V_MZ_ENC_PHZ: no longer IC3B.+IN
- net IN_3V3_MZ_ALARM: now also IC17D.OUT; no longer IC3C.OUT
- net IN_5V_GPI1_0V-30V: now also IC12D.OUT, J_ARD.32; no longer IC12B.OUT, J_ARD.27
- net IN_5V_GPI3_0V-30V: now also IC12B.OUT, J_ARD.27; no longer IC13A.OUT, J_ARD.29
- net IN_5V_GPI4_0V-30V: now also IC13A.OUT, J_ARD.29; no longer IC13C.OUT, J_ARD.30
- net IN_5V_GPI5_0V-30V: now also IC13B.OUT, J_ARD.33; no longer IC13D.OUT, J_ARD.31
- net IN_5V_GPI6_0V-30V: now also IC13C.OUT, J_ARD.30; no longer IC12D.OUT, J_ARD.32
- net IN_5V_GPI7_0V-30V: now also IC13D.OUT, J_ARD.31; no longer IC13B.OUT, J_ARD.33
- net N$32: now also IC1D.+IN; no longer IC2B.+IN
- net OUT_3V3_GPO1_H: now also J10.34, U7.1A4; no longer J9.10, U7.1A1
- net OUT_3V3_GPO2_H: now also J9.20, U7.1A3; no longer J9.11, U7.1A2
- net OUT_3V3_GPO3_H: now also J9.18, U7.1A2; no longer J9.14, U7.1A3
- net OUT_3V3_GPO4_H: now also U7.1A1; no longer U7.1A4
- net OUT_3V3_GPO5_H: now also J9.14, U7.2A2; no longer J9.18, U7.2A4
- net OUT_3V3_GPO6_H: now also J9.11; no longer J10.34
- net OUT_3V3_GPO7_H: now also J9.10, U7.2A4; no longer J9.20, U7.2A2
- net OUT_3V3_M1_CCW: now also J8/J6.7; no longer J8/J6.11
- net OUT_3V3_M2_CW: now also J8/J6.11; no longer J8/J6.7
- net OUT_5V_GPO1_H: now also U7.1Y4; no longer U7.1Y1
- net OUT_5V_GPO2_H: now also U7.1Y3; no longer U7.1Y2
- net OUT_5V_GPO3_H: now also U7.1Y2; no longer U7.1Y3
- net OUT_5V_GPO4_24V-5V: now also IC11D.+IN, J_ARD.23; no longer IC11A.+IN, J_ARD.20
- net OUT_5V_GPO4_H: now also U7.1Y1; no longer U7.1Y4
- net OUT_5V_GPO5_24V-5V: now also IC11A.+IN, J_ARD.20; no longer IC11B.+IN, J_ARD.21
- net OUT_5V_GPO5_H: now also U7.2Y2; no longer U7.2Y4
- net OUT_5V_GPO6_24V-5V: now also IC11B.+IN, J_ARD.21; no longer IC11C.+IN, J_ARD.22
- net OUT_5V_GPO7_24V-5V: now also IC11C.+IN, J_ARD.22; no longer IC11D.+IN, J_ARD.23
- net OUT_5V_GPO7_H: now also U7.2Y4; no longer U7.2Y2
- net VS_TEMP: now also IC1D.-IN, IC1D.OUT; no longer IC2B.-IN, IC2B.OUT
Other:
- moved on the sheet: IC1C, IC1D, U8

Commit message: 30/03/2021 fine primo routing
Parts:
- removed MOTZ_2: 61201021621, SCARA:61201021621
- added BRAKE, EMRG_CHN: CON_2F, SCARA:CON_2F
- renumbered MOTZ_1 to MOTZ
Connections:
- removed net IN_24V_MZ_ENC_CCW: MOTZ.5
- removed net IN_24V_MZ_ENC_CW: MOTZ.4
- removed net IN_24V_MZ_ENC_PHZ: MOTZ.6
- removed net N$30: J5/J7.10
- net +3V3: now also EMRG_CHN.2
- net GND: now also BRAKE.2
- net IN_24V_MZ_ALARM: now also MOTZ.8; no longer MOTZ.7
- net IN_30V_EDGE1: now also IC15D.+IN; no longer IC15B.+IN
- net IN_30V_EDGE10: now also IC16C.+IN; no longer IC17C.+IN
- net IN_30V_EDGE3: now also IC15B.+IN; no longer IC15D.+IN
- net IN_30V_EDGE4: now also IC17A.+IN; no longer IC16A.+IN
- net IN_30V_EDGE5: now also IC17B.+IN; no longer IC16B.+IN
- net IN_30V_EDGE6: now also IC17C.+IN; no longer IC16C.+IN
- net IN_30V_EDGE7: now also IC16A.+IN; no longer IC16D.+IN
- net IN_30V_EDGE8: now also IC16B.+IN; no longer IC17A.+IN
- net IN_30V_EDGE9: now also IC16D.+IN; no longer IC17B.+IN
- net IN_3V3_EDGE1: now also IC15D.OUT; no longer IC15B.OUT
- net IN_3V3_EDGE10: now also IC16C.OUT; no longer IC17C.OUT
- net IN_3V3_EDGE2: now also J4/J2.11; no longer J4/J2.9
- net IN_3V3_EDGE3: now also IC15B.OUT, J4/J2.9; no longer IC15D.OUT, J4/J2.11
- net IN_3V3_EDGE4: now also IC17A.OUT; no longer IC16A.OUT
- net IN_3V3_EDGE5: now also IC17B.OUT, J9.24; no longer IC16B.OUT, J9.23
- net IN_3V3_EDGE6: now also IC17C.OUT, J9.23; no longer IC16C.OUT, J9.24
- net IN_3V3_EDGE7: now also IC16A.OUT; no longer IC16D.OUT
- net IN_3V3_EDGE8: now also IC16B.OUT; no longer IC17A.OUT
- net IN_3V3_EDGE9: now also IC16D.OUT; no longer IC17B.OUT
- net IN_3V3_EMRGN_CHN: now also EMRG_CHN.1
- net OUT_24V_MZ_DIR: now also MOTZ.7; no longer MOTZ.10
- net OUT_24V_MZ_IMP: now also MOTZ.6; no longer MOTZ.9
- net OUT_24V_MZ_TRIGGER: now also MOTZ.3; no longer MOTZ.8
- net OUT_3V3_MZ_DIR: now also J5/J7.17; no longer J8/J6.3
- net OUT_3V3_MZ_IMP: now also J8/J6.3; no longer J8/J6.1
- net OUT_3V3_MZ_TRIGGER: now also J8/J6.1; no longer J5/J7.17
- net OUT_M2_BRAKE: now also BRAKE.1
- net OUT_MZ_EN: now also MOTZ.9; no longer MOTZ.3
- net OUT_MZ_HOMING: now also MOTZ.10; no longer MOTZ_2.1
