File: Tesi/comando 24V.sch (EAGLE design)
At the start: 104 parts, among them IC1 LM324N, IC11 LM324N, IC12 LM324N, IC13 LM324N, IC14 LM324N, IC15 LM324N, IC16 LM324N, IC17 LM324N, IC5 LM324N, IC7 LM324N, J1 61201021621, J1/J3 61202021621, J10 SBH11-PBPC-D25-ST-BK, J2 61201021621, J3 61201021621, J4 61201021621, J4/J2 61202021621, J5 61201021621, J5/J7 61202021621, J6 61201021621, J7 61201021621, J8 61202021621, J8/J6 61202021621, J9 SBH11-PBPC-D25-ST-BK, U1 ULN2003A, U2 ULN2003A, U3 TMP37FT9Z, U4 SN74LS244N, U5 SN74LS244N, U6 SN74LS244N, U7 SN74LS244N, U8 H11L1M

Commit message: 11/05/2021 mattina
Parts:
- R14, R16, R18, R25, R27: value 47k -> 22K
- R20, R21, R22, R23, R24: value 4k7 -> 3K
Changed lines of the file:
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@@
 <setting verticaltext="up"/>
 </settings>
-<grid distance="0.05" unitdist="inch" unit="inch" style="lines" multiple="1" display="no" altdistance="0.01" altunitdist="inch" altunit="inch"/>
+<grid distance="0.1" unitdist="inch" unit="inch" style="lines" multiple="1" display="no" altdistance="0.01" altunitdist="inch" altunit="inch"/>
 <layers>
 <layer number="1" name="Top" color="4" fill="1" visible="no" active="no"/>
@@
 <part name="FRAME5" library="frames" library_urn="urn:adsk.eagle:library:229" deviceset="A4L-LOC" device=""/>
 <part name="FRAME6" library="frames" library_urn="urn:adsk.eagle:library:229" deviceset="A4L-LOC" device=""/>
-<part name="R16" library="SCARA" deviceset="R-EU_207/10" device="0207/10" package3d_urn="urn:adsk.eagle:package:23491/2" value="47k"/>
+<part name="R16" library="SCARA" deviceset="R-EU_207/10" device="0207/10" package3d_urn="urn:adsk.eagle:package:23491/2" value="22K"/>
 <part name="R17" library="SCARA" deviceset="64WR5KLF" device="" value="TEMP_ADJ"/>
 <part name="P+3" library="supply1" library_urn="urn:adsk.eagle:library:371" deviceset="+24V" device=""/>
@@
 <part name="EN_IN_ENC" library="SCARA" deviceset="STRIP_3" device=""/>
 <part name="IC5" library="SCARA" deviceset="LM324" device="N" package3d_urn="urn:adsk.eagle:package:16407/2"/>
-<part name="R18" library="SCARA" deviceset="R-EU_207/10" device="0207/10" package3d_urn="urn:adsk.eagle:package:23491/2" value="47k"/>
+<part name="R18" library="SCARA" deviceset="R-EU_207/10" device="0207/10" package3d_urn="urn:adsk.eagle:package:23491/2" value="22K"/>
 <part name="R19" library="SCARA" deviceset="64WR5KLF" device="" value="VS_3V3_ADJ"/>
 <part name="P+4" library="supply1" library_urn="urn:adsk.eagle:library:371" deviceset="+24V" device=""/>
@@
 <part name="IC7" library="SCARA" deviceset="LM324" device="N" package3d_urn="urn:adsk.eagle:package:16407/2"/>
 <part name="IC11" library="SCARA" deviceset="LM324" device="N" package3d_urn="urn:adsk.eagle:package:16407/2"/>
-<part name="R14" library="SCARA" deviceset="R-EU_207/10" device="0207/10" package3d_urn="urn:adsk.eagle:package:23491/2" value="47k"/>
+<part name="R14" library="SCARA" deviceset="R-EU_207/10" device="0207/10" package3d_urn="urn:adsk.eagle:package:23491/2" value="22K"/>
 <part name="R15" library="SCARA" deviceset="64WR5KLF" device="" value="VS_5v_ADJ"/>
 <part name="P+5" library="supply1" library_urn="urn:adsk.eagle:library:371" deviceset="+24V" device=""/>
@@
 <part name="EN_M2_ENC_PHZ" library="SCARA" deviceset="STRIP_2" device=""/>
 <part name="EN_M1_ENC_PHZ" library="SCARA" deviceset="STRIP_2" device=""/>
-<part name="R20" library="SCARA" deviceset="R-EU_207/10" device="0207/10" package3d_urn="urn:adsk.eagle:package:23491/2" value="4k7"/>
-<part name="R21" library="SCARA" deviceset="R-EU_207/10" device="0207/10" package3d_urn="urn:adsk.eagle:package:23491/2" value="4k7"/>
-<part name="R22" library="SCARA" deviceset="R-EU_207/10" device="0207/10" package3d_urn="urn:adsk.eagle:package:23491/2" value="4k7"/>
-<part name="R23" library="SCARA" deviceset="R-EU_207/10" device="0207/10" package3d_urn="urn:adsk.eagle:package:23491/2" value="4k7"/>
-<part name="R24" library="SCARA" deviceset="R-EU_207/10" device="0207/10" package3d_urn="urn:adsk.eagle:package:23491/2" value="4k7"/>
+<part name="R20" library="SCARA" deviceset="R-EU_207/10" device="0207/10" package3d_urn="urn:adsk.eagle:package:23491/2" value="3K"/>
+<part name="R21" library="SCARA" deviceset="R-EU_207/10" device="0207/10" package3d_urn="urn:adsk.eagle:package:23491/2" value="3K"/>
+<part name="R22" library="SCARA" deviceset="R-EU_207/10" device="0207/10" package3d_urn="urn:adsk.eagle:package:23491/2" value="3K"/>
+<part name="R23" library="SCARA" deviceset="R-EU_207/10" device="0207/10" package3d_urn="urn:adsk.eagle:package:23491/2" value="3K"/>
+<part name="R24" library="SCARA" deviceset="R-EU_207/10" device="0207/10" package3d_urn="urn:adsk.eagle:package:23491/2" value="3K"/>
 <part name="FRAME2" library="frames" library_urn="urn:adsk.eagle:library:229" deviceset="A4L-LOC" device=""/>
 <part name="IC12" library="SCARA" deviceset="LM324" device="N" package3d_urn="urn:adsk.eagle:package:16407/2"/>
 <part name="IC13" library="SCARA" deviceset="LM324" device="N" package3d_urn="urn:adsk.eagle:package:16407/2"/>
 <part name="IC14" library="SCARA" deviceset="LM324" device="N" package3d_urn="urn:adsk.eagle:package:16407/2"/>
-<part name="R25" library="SCARA" deviceset="R-EU_207/10" device="0207/10" package3d_urn="urn:adsk.eagle:package:23491/2" value="47k"/>
+<part name="R25" library="SCARA" deviceset="R-EU_207/10" device="0207/10" package3d_urn="urn:adsk.eagle:package:23491/2" value="22K"/>
 <part name="R26" library="SCARA" deviceset="64WR5KLF" device="" value="VS_ARD_ADJ"/>
 <part name="P+2" library="supply1" library_urn="urn:adsk.eagle:library:371" deviceset="+24V" device=""/>
@@
 <part name="IC16" library="SCARA" deviceset="LM324" device="N" package3d_urn="urn:adsk.eagle:package:16407/2"/>
 <part name="IC17" library="SCARA" deviceset="LM324" device="N" package3d_urn="urn:adsk.eagle:package:16407/2"/>
-<part name="R27" library="SCARA" deviceset="R-EU_207/10" device="0207/10" package3d_urn="urn:adsk.eagle:package:23491/2" value="47k"/>
+<part name="R27" library="SCARA" deviceset="R-EU_207/10" device="0207/10" package3d_urn="urn:adsk.eagle:package:23491/2" value="22K"/>
 <part name="R28" library="SCARA" deviceset="64WR5KLF" device="" value="VS_EDGE_ADJ"/>
 <part name="P+6" library="supply1" library_urn="urn:adsk.eagle:library:371" deviceset="+24V" device=""/>
