File: Tesi/comando 24V.brd (EAGLE design)
At the start: 226.1 x 133.9 mm, 108 parts, among them IC1 LM324N, IC11 LM324N, IC12 LM324N, IC13 LM324N, IC14 LM324N, IC15 LM324N, IC16 LM324N, IC17 LM324N, IC2 LM324N, IC3 LM324N, IC5 LM324N, IC7 LM324N, J1 61201021621, J1/J3 61202021621, J10 SBH11-PBPC-D25-ST-BK, J2 61201021621, J3 61201021621, J4 61201021621, J4/J2 61202021621, J5 61201021621, J5/J7 61202021621, J6 61201021621, J7 61201021621, J8 61202021621, J8/J6 61202021621, J9 SBH11-PBPC-D25-ST-BK, U1 ULN2003A, U2 ULN2003A, U3 TMP37FT9Z, U4 SN74LS244N, U5 SN74LS244N, U6 SN74LS244N, U7 SN74LS244N, U8 H11L1M

Commit message: 23/03/2021 placing
Parts:
- added C1: UMF1V010MDD1TP, SCARA:UM-B_NCH
- moved IC5 44.7 mm to (17.0, 64.1)
- moved R16 40.0 mm to (64.1, 64.5)
- moved R17 40.0 mm to (70.5, 62.0)
- moved R27 40.0 mm to (50.2, 64.5)
- moved R28 40.0 mm to (57.8, 62.0)
- moved J_GPO/I2C_H1 37.6 mm to (91.9, 80.4)
- moved JI_TEXAS 16.7 mm to (38.1, 88.9), turned to 0 degrees
- moved R13 15.2 mm to (143.5, 85.1)
- moved R24 15.2 mm to (147.3, 85.1)
- moved U$12 15.2 mm to (143.5, 76.2)
- moved SUP_3V3 12.3 mm to (96.3, 101.2)
- moved SUP_5V 12.3 mm to (79.8, 101.2)
- moved R11 7.62 mm to (151.1, 85.1)
- moved R12 7.62 mm to (158.8, 85.1)
- moved R22 7.62 mm to (154.9, 85.1)
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Connections:
- net +24V: now also C1.1
- net GND: now also C1.2
Routing:
- net GND: track 1187.9 -> 0.00 mm, vias 1 -> 0
- net +5V: track 644.7 -> 0.00 mm, vias 4 -> 0
- net +24V: track 618.4 -> 0.00 mm, vias 4 -> 0
- net OUT_M1_BKW_INIB: track 259.0 -> 0.00 mm, vias 2 -> 0
- net +3V3: track 253.0 -> 0.00 mm, vias 2 -> 0
- net IN_3V3_M2_ALARM: track 222.1 -> 0.00 mm
- net OUT_M1_FWD_INIB: track 210.0 -> 0.00 mm, vias 1 -> 0
- net OUT_MZ_EN: track 205.7 -> 0.00 mm, vias 1 -> 0
- net IN_5V_M2_ENC_PHB: track 201.9 -> 0.00 mm, vias 3 -> 0
- net IN_5V_M2_ENC_PHZ: track 194.4 -> 0.00 mm, vias 3 -> 0
- net OUT_MZ_HOMING: track 183.8 -> 0.00 mm, vias 2 -> 0
- net IN_24V_HOMING_SENS_M2: track 181.3 -> 0.00 mm
- net OUT_M1_RUN: track 181.1 -> 0.00 mm, vias 2 -> 0
- net IN_5V_M2_ENC_PHA: track 180.9 -> 0.00 mm, vias 1 -> 0
- net IN_3V3_220V_ALARM: track 178.8 -> 0.00 mm, vias 1 -> 0
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
Commit message: inizio routing
Parts:
- moved J8 1.54 mm to (182.8, 66.3)
- moved R14 0.23 mm to (165.2, 37.9), turned to 180 degrees
- moved R29 0.06 mm to (171.4, 127.0), turned to 90 degrees
Connections:
- net IN_3V3_M1_ENC_PHA renamed IN_3V3_M1_ENC_PH_P
- net IN_3V3_M1_ENC_PHB renamed IN_3V3_M1_ENC_PH_N
- net IN_3V3_M2_ENC_PHA renamed IN_3V3_M2_ENC_PH_P
- net IN_3V3_M2_ENC_PHB renamed IN_3V3_M2_ENC_PH_N
- net IN_5V_M1_ENC_PHA renamed IN_5V_M1_ENC_PH_P
- net IN_5V_M1_ENC_PHB renamed IN_5V_M1_ENC_PH_N
- net IN_5V_M2_ENC_PHA renamed IN_5V_M2_ENC_PH_P
- net IN_5V_M2_ENC_PHB renamed IN_5V_M2_ENC_PH_N
- removed net N$39: IC5.12, R18.1, R19.3
- new net N$25: IC12.3, R26.2
- new net N$27: IC7.12, R15.2
- new net N$29: IC5.12, R19.2
- new net N$31: R18.1, R19.1
- new net N$32: IC2.5, R17.2
- new net N$33: IC15.3, R28.2
- net GND: now also R15.3, R17.3, R19.3, R26.3, R28.3; no longer R15.1, R17.1, R19.1, R26.1, R28.1
- net IN_30V_GPI1: now also IC12.12; no longer IC12.5
- net IN_30V_GPI3: now also IC12.5; no longer IC12.12
- net IN_5V_GPI3_0V-30V: now also IC13.1; no longer IC12.14
- net IN_5V_GPI4_0V-30V: now also IC13.8; no longer IC13.1
- net IN_5V_GPI5_0V-30V: now also IC13.14; no longer IC13.7
- net IN_5V_GPI6_0V-30V: now also IC12.14; no longer IC13.8
- net IN_5V_GPI7_0V-30V: now also IC13.7; no longer IC13.14
- net N$14: now also R17.1; no longer IC2.5, R17.3
- net N$15: now also R26.1; no longer IC12.3, R26.3
- net N$17: now also R28.1; no longer IC15.3, R28.3
- net N$20: now also R15.1; no longer IC7.12, R15.3
- net OUT_24V-5V_GPO4: now also IC11.14; no longer IC11.1
- net OUT_24V-5V_GPO5: now also IC11.1; no longer IC11.7
- net OUT_24V-5V_GPO6: now also IC11.7; no longer IC11.8
- net OUT_24V-5V_GPO7: now also IC11.8; no longer IC11.14
- net OUT_5V_M1_CCW_INIB: now also J_ARD.6; no longer J_ARD.7
- net OUT_5V_M1_CW_INIB: now also J_ARD.7; no longer J_ARD.6
- net OUT_5V_M2_CCW_INIB: now also J_ARD.8; no longer J_ARD.9
- net OUT_5V_M2_CW_INIB: now also J_ARD.9; no longer J_ARD.8
Routing:
- net +5V: track 0.00 -> 561.2 mm, vias 0 -> 3
- net +24V: track 0.00 -> 541.9 mm, vias 0 -> 3
- net +3V3: track 0.00 -> 237.0 mm, vias 0 -> 4
- net IN_5V_M2_ENC_PH_N: track 0.00 -> 203.6 mm
- net IN_5V_M2_ENC_PH_P: track 0.00 -> 197.1 mm
- net IN_5V_M1_ENC_PH_P: track 0.00 -> 141.7 mm, vias 0 -> 1
- net IN_5V_M1_ENC_PH_N: track 0.00 -> 137.7 mm, vias 0 -> 1
- net IN_3V3_M2_ENC_PH_P: track 0.00 -> 126.4 mm, vias 0 -> 1
- net IN_3V3_M2_ENC_PH_N: track 0.00 -> 118.6 mm
- net IN_3V3_M1_ENC_PH_P: track 0.00 -> 108.1 mm
- net IN_3V3_M1_ENC_PH_N: track 0.00 -> 106.1 mm
- net VS_IN_ARD: track 0.00 -> 96.4 mm, vias 0 -> 3
- net IN_3V3_SCI_RX: track 0.00 -> 62.5 mm
- net OUT_3V3_SCI_TX: track 0.00 -> 56.0 mm
- net OUT_5V_GPO7_24V-5V: track 0.00 -> 55.1 mm, vias 0 -> 1
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
Commit message: 28/03/2021
Parts:
- removed C1: UMF1V010MDD1TP, SCARA:UM-B_NCH
- removed IC2: LM324N, linear:DIL14
- removed IC3: LM324N, SCARA:DIL14
- added C2: QYX1H102JTP3TA, SCARA:CAP_QYX_2P5X5X8P5_NCH
- added C3: UBY2A301MHL, SCARA:CAP_UBY_12P5X31P5_NCH
- moved R1 32.3 mm to (154.2, 63.4)
- moved U$1 32.3 mm to (154.2, 54.6)
- moved R7 31.8 mm to (121.9, 63.4)
- moved U$6 31.8 mm to (121.9, 54.6)
- moved R21 24.1 mm to (163.8, 85.1)
- moved U$9 23.7 mm to (159.6, 76.2)
- moved R10 23.7 mm to (159.6, 85.1)
- moved R2 19.4 mm to (147.7, 63.4)
- moved U$2 19.4 mm to (147.7, 54.6)
- moved R6 19.0 mm to (128.3, 63.4)
- moved U$5 19.0 mm to (128.3, 54.6)
- moved R12 15.9 mm to (142.8, 85.1)
- moved R23 15.6 mm to (147.0, 85.1)
- moved U$11 14.2 mm to (144.5, 76.2)
- moved R13 9.07 mm to (134.4, 85.1)
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Connections:
- removed net IN_3V3_MZ_ENC_CCW: IC3.1
- removed net IN_3V3_MZ_ENC_CW: IC1.14
- removed net IN_3V3_MZ_ENC_PHZ: IC3.7
- net +24V: now also C2.1, C3.1; no longer C1.1
- net +3V3: now also IC17.13; no longer IC1.13, IC3.2, IC3.6, IC3.9
- net +5V: no longer IC2.4, IC3.4
- net GND: now also C2.2, C3.2; no longer C1.2, IC2.11, IC3.11
- net IN_24V_MZ_ALARM: now also IC17.12; no longer IC3.10
- net IN_24V_MZ_ENC_CCW: no longer IC3.3
- net IN_24V_MZ_ENC_CW: no longer IC1.12
- net IN_24V_MZ_ENC_PHZ: no longer IC3.5
- net IN_3V3_MZ_ALARM: now also IC17.14; no longer IC3.8
- net IN_5V_GPI1_0V-30V: now also IC12.14, J_ARD.32; no longer IC12.7, J_ARD.27
- net IN_5V_GPI3_0V-30V: now also IC12.7, J_ARD.27; no longer IC13.1, J_ARD.29
- net IN_5V_GPI4_0V-30V: now also IC13.1, J_ARD.29; no longer IC13.8, J_ARD.30
- net IN_5V_GPI5_0V-30V: now also IC13.7, J_ARD.33; no longer IC13.14, J_ARD.31
- net IN_5V_GPI6_0V-30V: now also IC13.8, J_ARD.30; no longer IC12.14, J_ARD.32
- net IN_5V_GPI7_0V-30V: now also IC13.14, J_ARD.31; no longer IC13.7, J_ARD.33
- net N$32: now also IC1.12; no longer IC2.5
- net OUT_3V3_GPO1_H: now also J10.34, U7.8; no longer J9.10, U7.2
- net OUT_3V3_GPO2_H: now also J9.20, U7.6; no longer J9.11, U7.4
- net OUT_3V3_GPO3_H: now also J9.18, U7.4; no longer J9.14, U7.6
- net OUT_3V3_GPO4_H: now also U7.2; no longer U7.8
- net OUT_3V3_GPO5_H: now also J9.14, U7.13; no longer J9.18, U7.17
- net OUT_3V3_GPO6_H: now also J9.11; no longer J10.34
- net OUT_3V3_GPO7_H: now also J9.10, U7.17; no longer J9.20, U7.13
- net OUT_3V3_M1_CCW: now also J8/J6.4; no longer J8/J6.6
- net OUT_3V3_M2_CW: now also J8/J6.6; no longer J8/J6.4
- net OUT_5V_GPO1_H: now also U7.12; no longer U7.18
- net OUT_5V_GPO2_H: now also U7.14; no longer U7.16
- net OUT_5V_GPO3_H: now also U7.16; no longer U7.14
- net OUT_5V_GPO4_24V-5V: now also IC11.12, J_ARD.23; no longer IC11.3, J_ARD.20
- net OUT_5V_GPO4_H: now also U7.18; no longer U7.12
- net OUT_5V_GPO5_24V-5V: now also IC11.3, J_ARD.20; no longer IC11.5, J_ARD.21
- net OUT_5V_GPO5_H: now also U7.7; no longer U7.3
- net OUT_5V_GPO6_24V-5V: now also IC11.5, J_ARD.21; no longer IC11.10, J_ARD.22
- net OUT_5V_GPO7_24V-5V: now also IC11.10, J_ARD.22; no longer IC11.12, J_ARD.23
- net OUT_5V_GPO7_H: now also U7.3; no longer U7.7
- net VS_TEMP: now also IC1.13, IC1.14; no longer IC2.6, IC2.7
Routing:
- net OUT_M1_RUN: track 0.00 -> 222.3 mm, vias 0 -> 7
- net OUT_M2_FWD_INIB: track 0.00 -> 159.8 mm, vias 0 -> 4
- net OUT_24V_ELVALV: track 0.00 -> 140.1 mm
- net OUT_24V_GPO2: track 0.00 -> 132.4 mm
- net OUT_M2_RUN: track 0.00 -> 130.9 mm, vias 0 -> 4
- net OUT_24V_GPO1: track 0.00 -> 126.4 mm
- net OUT_M2_BKW_INIB: track 0.00 -> 124.7 mm, vias 0 -> 3
- net OUT_MZ_HOMING: track 0.00 -> 74.4 mm
- net OUT_MZ_EN: track 0.00 -> 74.3 mm
- net I/O_3V3_I2C_SCL: track 0.00 -> 71.4 mm
- net I/O_3V3_I2C_SDA: track 0.00 -> 69.7 mm
- net VS_5V: track 0.00 -> 65.2 mm, vias 0 -> 1
- net IN_3V3_HOMING_SENS_M1: track 0.00 -> 62.4 mm, vias 0 -> 2
- net OUT_M1_FWD_INIB: track 0.00 -> 58.6 mm, vias 0 -> 2
- net IN_3V3_HOMING_SENS_M2: track 0.00 -> 52.9 mm, vias 0 -> 2
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
Commit message: 30/03/2021 fine primo routing
Parts:
- removed MOTZ_2: 61201021621, SCARA:CONN_61201021621_WRE
- added BRAKE, EMRG_CHN: CON_2F, SCARA:CON_2F
- moved EL_VALV 11.9 mm to (217.2, 51.6)
- moved PROXYM_M1 11.9 mm to (217.2, 32.5)
- moved PROXYM_M2 11.9 mm to (217.2, 13.5)
- moved U$17 10.0 mm to (221.7, 5.12)
- renumbered MOTZ_1 to MOTZ
Connections:
- removed net IN_24V_MZ_ENC_CCW: MOTZ.5
- removed net IN_24V_MZ_ENC_CW: MOTZ.4
- removed net IN_24V_MZ_ENC_PHZ: MOTZ.6
- removed net N$30: J5/J7.15
- net +3V3: now also EMRG_CHN.2
- net GND: now also BRAKE.2
- net IN_24V_MZ_ALARM: now also MOTZ.8; no longer MOTZ.7
- net IN_30V_EDGE1: now also IC15.12; no longer IC15.5
- net IN_30V_EDGE10: now also IC16.10; no longer IC17.10
- net IN_30V_EDGE3: now also IC15.5; no longer IC15.12
- net IN_30V_EDGE4: now also IC17.3; no longer IC16.3
- net IN_30V_EDGE5: now also IC17.5; no longer IC16.5
- net IN_30V_EDGE6: now also IC17.10; no longer IC16.10
- net IN_30V_EDGE7: now also IC16.3; no longer IC16.12
- net IN_30V_EDGE8: now also IC16.5; no longer IC17.3
- net IN_30V_EDGE9: now also IC16.12; no longer IC17.5
- net IN_3V3_EDGE1: now also IC15.14; no longer IC15.7
- net IN_3V3_EDGE10: now also IC16.8; no longer IC17.8
- net IN_3V3_EDGE2: now also J4/J2.6; no longer J4/J2.5
- net IN_3V3_EDGE3: now also IC15.7, J4/J2.5; no longer IC15.14, J4/J2.6
- net IN_3V3_EDGE4: now also IC17.1; no longer IC16.1
- net IN_3V3_EDGE5: now also IC17.7, J9.24; no longer IC16.7, J9.23
- net IN_3V3_EDGE6: now also IC17.8, J9.23; no longer IC16.8, J9.24
- net IN_3V3_EDGE7: now also IC16.1; no longer IC16.14
- net IN_3V3_EDGE8: now also IC16.7; no longer IC17.1
- net IN_3V3_EDGE9: now also IC16.14; no longer IC17.7
- net IN_3V3_EMRGN_CHN: now also EMRG_CHN.1
- net OUT_24V_MZ_DIR: now also MOTZ.7; no longer MOTZ.10
- net OUT_24V_MZ_IMP: now also MOTZ.6; no longer MOTZ.9
- net OUT_24V_MZ_TRIGGER: now also MOTZ.3; no longer MOTZ.8
- net OUT_3V3_MZ_DIR: now also J5/J7.9; no longer J8/J6.2
- net OUT_3V3_MZ_IMP: now also J8/J6.2; no longer J8/J6.1
- net OUT_3V3_MZ_TRIGGER: now also J8/J6.1; no longer J5/J7.9
- net OUT_M2_BRAKE: now also BRAKE.1
- net OUT_MZ_EN: now also MOTZ.9; no longer MOTZ.3
- net OUT_MZ_HOMING: now also MOTZ.10; no longer MOTZ_2.1
Routing:
- net IN_3V3_M1_ALARM: track 0.00 -> 267.8 mm
- net IN_24V_HOMING_SENS_M1: track 0.00 -> 260.6 mm, vias 0 -> 4
- net IN_3V3_EMRGN_CHN: track 0.00 -> 248.2 mm, vias 0 -> 1
- net IN_3V3_M2_ALARM: track 0.00 -> 241.5 mm, vias 0 -> 11
- net IN_3V3_M1_READY: track 0.00 -> 238.2 mm, vias 0 -> 1
- net IN_3V3_M2_READY: track 0.00 -> 215.0 mm, vias 0 -> 8
- net IN_5V_M2_ENC_PHZ: track 0.00 -> 189.2 mm, vias 0 -> 2
- net IN_24V_HOMING_SENS_M2: track 0.00 -> 182.6 mm, vias 0 -> 4
- net OUT_M1_FWD_INIB: track 58.6 -> 227.8 mm, vias 2 -> 9
- net IN_3V3_220V_ALARM: track 0.00 -> 167.7 mm, vias 0 -> 1
- net OUT_M1_BKW_INIB: track 51.2 -> 214.1 mm, vias 3 -> 7
- net IN_5V_M1_ENC_PHZ: track 0.00 -> 158.2 mm, vias 0 -> 1
- net OUT_5V_M1_CCW: track 0.00 -> 155.3 mm, vias 0 -> 1
- net OUT_MZ_HOMING: track 74.4 -> 219.5 mm
- net OUT_5V_M1_CW: track 0.00 -> 140.6 mm, vias 0 -> 1
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
Commit message: 06/04/2021 revisione frassine
Parts:
- moved PT1 5.06 mm to (216.2, 105.2)
- moved R5 4.32 mm to (207.8, 94.1)
Routing:
- net I/O_M2_33: track 0.00 -> 22.8 mm, vias 0 -> 1
- net N$18: track 0.00 -> 16.6 mm
- net N$9: track 16.2 -> 21.1 mm
- net 220V_PROBE: track 22.1 -> 17.3 mm
- net IN_3V3_MZ_ALARM: track 135.3 -> 133.0 mm, vias 1 -> 3
- net N$23: track 13.8 -> 12.0 mm
- net GND_220V: track 53.6 -> 55.5 mm
- net VS_IN_ARD: track 96.4 -> 97.5 mm
- net +5V: track 562.0 -> 563.0 mm
- net IN_3V3_M2_ENC_PH_N: track 118.6 -> 119.5 mm, vias 0 -> 2
- net IN_3V3_EDGE10: track 72.9 -> 73.1 mm, vias 2 -> 6
- net IN_3V3_EDGE6: track 87.5 -> 87.6 mm, vias 2 -> 4
- net N$33: vias 1 -> 0
- added copper zone on layer 1, net GND
- added copper zone on layer 16, net GND
