File: Tesi/comando 24V.brd (EAGLE design)
At the start: 226.1 x 133.9 mm, 109 parts, among them IC1 LM324N, IC11 LM324N, IC12 LM324N, IC13 LM324N, IC14 LM324N, IC15 LM324N, IC16 LM324N, IC17 LM324N, IC5 LM324N, IC7 LM324N, J1 61201021621, J1/J3 61202021621, J10 SBH11-PBPC-D25-ST-BK, J2 61201021621, J3 61201021621, J4 61201021621, J4/J2 61202021621, J5 61201021621, J5/J7 61202021621, J6 61201021621, J7 61201021621, J8 61202021621, J8/J6 61202021621, J9 SBH11-PBPC-D25-ST-BK, U1 ULN2003A, U2 ULN2003A, U3 TMP37FT9Z, U4 SN74LS244N, U5 SN74LS244N, U6 SN74LS244N, U7 SN74LS244N, U8 H11L1M

Commit message: messo a posto i drill files
Parts:
- R1, R10, R11, R12, R13, R14, R16, R18, R2, R20, R21, R22, R23, R24, R25, R27, R29, R3, R4, R6, R7, R8, R9: device rcl:0207/10 -> SCARA:0207/10

Commit message: 15/04/2021 avanzamento parser
Routing:
- removed copper zone on layer 16, net GND

Commit message: 11/05/2021 mattina
Parts:
- R14, R16, R18, R25, R27: value 47k -> 22K
- R20, R21, R22, R23, R24: value 4k7 -> 3K
Changed lines of the file:
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@@
 <attribute name="VALUE" x="135.07020625" y="82.8294" size="1.27" layer="27" ratio="10" rot="R90"/>
 </element>
-<element name="R14" library="SCARA" package="0207/10" package3d_urn="urn:adsk.eagle:package:23491/2" value="47k" x="165.1508" y="37.8714" smashed="yes" rot="R180">
+<element name="R14" library="SCARA" package="0207/10" package3d_urn="urn:adsk.eagle:package:23491/2" value="22K" x="165.1508" y="37.8714" smashed="yes" rot="R180">
 <attribute name="NAME" x="168.1988" y="36.3474" size="1.27" layer="25" ratio="10" rot="R180"/>
 <attribute name="POPULARITY" value="81" x="31.8008" y="206.7814" size="1.778" layer="27" rot="R180" display="off"/>
@@
 <attribute name="VENDOR" value="TT Electronics" x="245.11" y="-125.73" size="1.778" layer="27" display="off"/>
 </element>
-<element name="R16" library="SCARA" package="0207/10" package3d_urn="urn:adsk.eagle:package:23491/2" value="47k" x="64.13" y="64.5" smashed="yes" rot="R90">
+<element name="R16" library="SCARA" package="0207/10" package3d_urn="urn:adsk.eagle:package:23491/2" value="22K" x="64.13" y="64.5" smashed="yes" rot="R90">
 <attribute name="NAME" x="62.606" y="61.452" size="1.27" layer="25" ratio="10" rot="R90"/>
 <attribute name="POPULARITY" value="81" x="233.04" y="210.55" size="1.778" layer="27" rot="R90" display="off"/>
@@
 <attribute name="VENDOR" value="TT Electronics" x="233.04" y="144.51" size="1.778" layer="27" rot="R90" display="off"/>
 </element>
-<element name="R18" library="SCARA" package="0207/10" package3d_urn="urn:adsk.eagle:package:23491/2" value="47k" x="32.83" y="64.5" smashed="yes" rot="R90">
+<element name="R18" library="SCARA" package="0207/10" package3d_urn="urn:adsk.eagle:package:23491/2" value="22K" x="32.83" y="64.5" smashed="yes" rot="R90">
 <attribute name="NAME" x="31.306" y="61.452" size="1.27" layer="25" ratio="10" rot="R90"/>
 <attribute name="POPULARITY" value="81" x="201.74" y="223.25" size="1.778" layer="27" rot="R90" display="off"/>
@@
 <attribute name="VALUE" x="148.3514125" y="61.1886" size="1.27" layer="27" ratio="10" rot="R90"/>
 </element>
-<element name="R20" library="SCARA" package="0207/10" package3d_urn="urn:adsk.eagle:package:23491/2" value="4k7" x="130.2468375" y="85.09" smashed="yes" rot="R90">
+<element name="R20" library="SCARA" package="0207/10" package3d_urn="urn:adsk.eagle:package:23491/2" value="3K" x="130.2468375" y="85.09" smashed="yes" rot="R90">
 <attribute name="NAME" x="128.7228375" y="82.042" size="1.27" layer="25" ratio="10" rot="R90"/>
 <attribute name="POPULARITY" value="81" x="304.2368375" y="104.14" size="1.778" layer="27" rot="R90" display="off"/>
@@
 <attribute name="VALUE" x="130.8818375" y="82.8294" size="1.27" layer="27" ratio="10" rot="R90"/>
 </element>
-<element name="R21" library="SCARA" package="0207/10" package3d_urn="urn:adsk.eagle:package:23491/2" value="4k7" x="163.7537875" y="85.09" smashed="yes" rot="R90">
+<element name="R21" library="SCARA" package="0207/10" package3d_urn="urn:adsk.eagle:package:23491/2" value="3K" x="163.7537875" y="85.09" smashed="yes" rot="R90">
 <attribute name="NAME" x="162.2297875" y="82.042" size="1.27" layer="25" ratio="10" rot="R90"/>
 <attribute name="POPULARITY" value="81" x="337.7437875" y="116.84" size="1.778" layer="27" rot="R90" display="off"/>
@@
 <attribute name="VALUE" x="164.3887875" y="82.8294" size="1.27" layer="27" ratio="10" rot="R90"/>
 </element>
-<element name="R22" library="SCARA" package="0207/10" package3d_urn="urn:adsk.eagle:package:23491/2" value="4k7" x="155.37705" y="85.09" smashed="yes" rot="R90">
+<element name="R22" library="SCARA" package="0207/10" package3d_urn="urn:adsk.eagle:package:23491/2" value="3K" x="155.37705" y="85.09" smashed="yes" rot="R90">
 <attribute name="NAME" x="153.85305" y="82.042" size="1.27" layer="25" ratio="10" rot="R90"/>
 <attribute name="POPULARITY" value="81" x="329.36705" y="129.54" size="1.778" layer="27" rot="R90" display="off"/>
@@
 <attribute name="VALUE" x="156.01205" y="82.8294" size="1.27" layer="27" ratio="10" rot="R90"/>
 </element>
-<element name="R23" library="SCARA" package="0207/10" package3d_urn="urn:adsk.eagle:package:23491/2" value="4k7" x="147.0003125" y="85.09" smashed="yes" rot="R90">
+<element name="R23" library="SCARA" package="0207/10" package3d_urn="urn:adsk.eagle:package:23491/2" value="3K" x="147.0003125" y="85.09" smashed="yes" rot="R90">
 <attribute name="NAME" x="145.4763125" y="82.042" size="1.27" layer="25" ratio="10" rot="R90"/>
 <attribute name="POPULARITY" value="81" x="320.9903125" y="142.24" size="1.778" layer="27" rot="R90" display="off"/>
@@
 <attribute name="VALUE" x="147.6353125" y="82.8294" size="1.27" layer="27" ratio="10" rot="R90"/>
 </element>
-<element name="R24" library="SCARA" package="0207/10" package3d_urn="urn:adsk.eagle:package:23491/2" value="4k7" x="138.623575" y="85.09" smashed="yes" rot="R90">
+<element name="R24" library="SCARA" package="0207/10" package3d_urn="urn:adsk.eagle:package:23491/2" value="3K" x="138.623575" y="85.09" smashed="yes" rot="R90">
 <attribute name="NAME" x="137.099575" y="82.042" size="1.27" layer="25" ratio="10" rot="R90"/>
 <attribute name="POPULARITY" value="81" x="312.613575" y="154.94" size="1.778" layer="27" rot="R90" display="off"/>
@@
 <attribute name="VALUE" x="139.258575" y="82.8294" size="1.27" layer="27" ratio="10" rot="R90"/>
 </element>
-<element name="R25" library="SCARA" package="0207/10" package3d_urn="urn:adsk.eagle:package:23491/2" value="47k" x="189.23" y="38.1" smashed="yes" rot="R180">
+<element name="R25" library="SCARA" package="0207/10" package3d_urn="urn:adsk.eagle:package:23491/2" value="22K" x="189.23" y="38.1" smashed="yes" rot="R180">
 <attribute name="NAME" x="192.278" y="36.576" size="1.27" layer="25" ratio="10" rot="R180"/>
 <attribute name="POPULARITY" value="81" x="106.68" y="212.09" size="1.778" layer="27" rot="R180" display="off"/>
@@
 <attribute name="VENDOR" value="TT Electronics" x="242.57" y="-125.73" size="1.778" layer="27" display="off"/>
 </element>
-<element name="R27" library="SCARA" package="0207/10" package3d_urn="urn:adsk.eagle:package:23491/2" value="47k" x="50.16" y="64.5" smashed="yes" rot="R90">
+<element name="R27" library="SCARA" package="0207/10" package3d_urn="urn:adsk.eagle:package:23491/2" value="22K" x="50.16" y="64.5" smashed="yes" rot="R90">
 <attribute name="NAME" x="48.636" y="61.452" size="1.27" layer="25" ratio="10" rot="R90"/>
 <attribute name="POPULARITY" value="81" x="224.15" y="159.75" size="1.778" layer="27" rot="R90" display="off"/>
